File: design/CAN.sch (KiCad schematic (older format))
At the start: 4 parts

Commit message: finished schematic and rename LESC to ESCX
Parts:
- gave numbers to parts that had none: 4
Changed lines of the file:
@@
 EESchema Schematic File Version 4
-LIBS:LESC-cache
+LIBS:ESCX-cache
 EELAYER 26 0
 EELAYER END
@@
 $EndDescr
 $Comp
-L crf_1:TJA1042TK_3 U?
+L crf_1:TJA1042TK_3 U6
 U 1 1 5AEABFE9
 P 5900 3200
-F 0 "U?" H 5900 3637 60  0000 C CNN
+F 0 "U6" H 5900 3637 60  0000 C CNN
 F 1 "TJA1042TK_3" H 5900 3531 60  0000 C CNN
 F 2 "" H 5900 3200 60  0000 C CNN
@@
 RX
 $Comp
-L Device:C C?
+L Device:C C41
 U 1 1 5AEAC294
 P 4600 3550
-F 0 "C?" H 4715 3596 50  0000 L CNN
+F 0 "C41" H 4715 3596 50  0000 L CNN
 F 1 "C" H 4715 3505 50  0000 L CNN
 F 2 "" H 4638 3400 50  0001 C CNN
@@
 $EndComp
 $Comp
-L Device:C C?
+L Device:C C42
 U 1 1 5AEAC2CC
 P 6900 3600
-F 0 "C?" H 7015 3646 50  0000 L CNN
+F 0 "C42" H 7015 3646 50  0000 L CNN
 F 1 "C" H 7015 3555 50  0000 L CNN
 F 2 "" H 6938 3450 50  0001 C CNN
@@
 	6900 3350 6900 3450
 $Comp
-L Device:R R?
+L Device:R R39
 U 1 1 5AEAC462
 P 7400 3200
-F 0 "R?" H 7470 3246 50  0000 L CNN
+F 0 "R39" H 7470 3246 50  0000 L CNN
 F 1 "R" H 7470 3155 50  0000 L CNN
 F 2 "" V 7330 3200 50  0001 C CNN

Commit message: add value
Parts:
- C44: renamed from C41; value C -> 2.2u
- C45: renamed from C42; value C -> 2.2u
- R39: value R -> 220R
- renumbered U6 to U7
Changed lines of the file:
@@
 encoding utf-8
 Sheet 5 7
-Title ""
-Date ""
-Rev ""
-Comp ""
+Title "VESC 6.4 redraw"
+Date "2018-06-03"
+Rev "6.4"
+Comp "LI XITONG"
 Comment1 ""
 Comment2 ""
@@
 $EndDescr
 $Comp
-L crf_1:TJA1042TK_3 U6
+L crf_1:TJA1042TK_3 U7
 U 1 1 5AEABFE9
 P 5900 3200
-F 0 "U6" H 5900 3637 60  0000 C CNN
+F 0 "U7" H 5900 3637 60  0000 C CNN
 F 1 "TJA1042TK_3" H 5900 3531 60  0000 C CNN
 F 2 "" H 5900 3200 60  0000 C CNN
@@
 RX
 $Comp
-L Device:C C41
+L Device:C C44
 U 1 1 5AEAC294
 P 4600 3550
-F 0 "C41" H 4715 3596 50  0000 L CNN
-F 1 "C" H 4715 3505 50  0000 L CNN
+F 0 "C44" H 4650 3650 50  0000 L CNN
+F 1 "2.2u" H 4650 3450 50  0000 L CNN
 F 2 "" H 4638 3400 50  0001 C CNN
 F 3 "~" H 4600 3550 50  0001 C CNN
@@
 $EndComp
 $Comp
-L Device:C C42
+L Device:C C45
 U 1 1 5AEAC2CC
 P 6900 3600
-F 0 "C42" H 7015 3646 50  0000 L CNN
-F 1 "C" H 7015 3555 50  0000 L CNN
+F 0 "C45" H 7000 3700 50  0000 L CNN
+F 1 "2.2u" H 7000 3500 50  0000 L CNN
 F 2 "" H 6938 3450 50  0001 C CNN
 F 3 "~" H 6900 3600 50  0001 C CNN
@@
 U 1 1 5AEAC462
 P 7400 3200
-F 0 "R39" H 7470 3246 50  0000 L CNN
-F 1 "R" H 7470 3155 50  0000 L CNN
+F 0 "R39" V 7500 3150 50  0000 L CNN
+F 1 "220R" V 7400 3100 50  0000 L CNN
 F 2 "" V 7330 3200 50  0001 C CNN
 F 3 "~" H 7400 3200 50  0001 C CNN

Commit message: finish sch
Parts:
- removed U7: TJA1042TK_3, symbol crf_1:TJA1042TK_3
- added U7: TJA1051TK-3, Package_DFN_QFN:DFN-8-1EP_3x3mm_P0.65mm_EP1.55x2.4mm, symbol bldc:TJA1051TK-3
- renumbered C44 to C48, C45 to C49
Connections:
- net labels added: +5V, GND, VCC
- wire segments 27 -> 32
Changed lines of the file:
@@
 Comment4 ""
 $EndDescr
-$Comp
-L crf_1:TJA1042TK_3 U7
-U 1 1 5AEABFE9
-P 5900 3200
-F 0 "U7" H 5900 3637 60  0000 C CNN
-F 1 "TJA1042TK_3" H 5900 3531 60  0000 C CNN
-F 2 "" H 5900 3200 60  0000 C CNN
-F 3 "" H 5900 3200 60  0000 C CNN
-	1    5900 3200
-	1    0    0    -1
-$EndComp
 Text HLabel 5300 3050 0    50   Input ~ 0
 TX
@@
 RX
 $Comp
-L Device:C C44
+L Device:C C48
 U 1 1 5AEAC294
 P 4600 3550
-F 0 "C44" H 4650 3650 50  0000 L CNN
+F 0 "C48" H 4650 3650 50  0000 L CNN
 F 1 "2.2u" H 4650 3450 50  0000 L CNN
 F 2 "" H 4638 3400 50  0001 C CNN
@@
 $EndComp
 $Comp
-L Device:C C45
+L Device:C C49
 U 1 1 5AEAC2CC
-P 6900 3600
-F 0 "C45" H 7000 3700 50  0000 L CNN
-F 1 "2.2u" H 7000 3500 50  0000 L CNN
-F 2 "" H 6938 3450 50  0001 C CNN
-F 3 "~" H 6900 3600 50  0001 C CNN
-	1    6900 3600
+P 6550 3600
+F 0 "C49" H 6650 3700 50  0000 L CNN
+F 1 "2.2u" H 6650 3500 50  0000 L CNN
+F 2 "" H 6588 3450 50  0001 C CNN
+F 3 "~" H 6550 3600 50  0001 C CNN
+	1    6550 3600
 	1    0    0    -1
 $EndComp
@@
 	4600 4000 4950 4000
 Wire Wire Line
-	6900 4000 6900 3750
+	6550 4000 6550 3750
 Wire Wire Line
 	5300 3150 4950 3150
@@
 Connection ~ 4950 4000
 Wire Wire Line
-	4950 4000 6650 4000
+	6150 3050 6300 3050
 Wire Wire Line
-	6500 3050 6650 3050
+	6300 3050 6300 4000
+Connection ~ 6300 4000
 Wire Wire Line
-	6650 3050 6650 4000
-Connection ~ 6650 4000
+	6300 4000 6550 4000
 Wire Wire Line
-	6650 4000 6900 4000
+	6150 3350 6550 3350
 Wire Wire Line
-	6500 3350 6900 3350
-Wire Wire Line
-	6900 3350 6900 3450
+	6550 3350 6550 3450
 $Comp
 L Device:R R39
 U 1 1 5AEAC462
-P 7400 3200
-F 0 "R39" V 7500 3150 50  0000 L CNN
-F 1 "220R" V 7400 3100 50  0000 L CNN
-F 2 "" V 7330 3200 50  0001 C CNN
-F 3 "~" H 7400 3200 50  0001 C CNN
-	1    7400 3200
+P 7050 3200
+F 0 "R39" V 7150 3150 50  0000 L CNN
+F 1 "220R" V 7050 3100 50  0000 L CNN
+F 2 "" V 6980 3200 50  0001 C CNN
+F 3 "~" H 7050 3200 50  0001 C CNN
+	1    7050 3200
 	1    0    0    -1
 $EndComp
 Wire Wire Line
-	6500 3250 7200 3250
+	6150 3250 6850 3250
 Wire Wire Line
-	7200 3250 7200 3450
+	6850 3250 6850 3450
 Wire Wire Line
-	7200 3450 7400 3450
+	6850 3450 7050 3450
 Wire Wire Line
-	7650 3450 7650 3250
+	7300 3450 7300 3250
 Wire Wire Line
-	7650 3250 7800 3250
+	7300 3250 7450 3250
 Wire Wire Line
-	6500 3150 7200 3150
+	6150 3150 6850 3150
 Wire Wire Line
-	7200 3150 7200 2900
+	6850 3150 6850 2900
 Wire Wire Line
-	7200 2900 7400 2900
+	6850 2900 7050 2900
 Wire Wire Line
-	7650 2900 7650 3100
+	7300 2900 7300 3100
 Wire Wire Line
-	7650 3100 7800 3100
+	7300 3100 7450 3100
 Wire Wire Line
-	7400 2900 7400 3050
-Connection ~ 7400 2900
+	7050 2900 7050 3050
+Connection ~ 7050 2900
 Wire Wire Line
-	7400 2900 7650 2900
+	7050 2900 7300 2900
 Wire Wire Line
-	7400 3350 7400 3450
-Connection ~ 7400 3450
+	7050 3350 7050 3450
+Connection ~ 7050 3450
 Wire Wire Line
-	7400 3450 7650 3450
-Text HLabel 7800 3100 2    50   Input ~ 0
+	7050 3450 7300 3450
+Text HLabel 7450 3100 2    50   Input ~ 0
 CANH
-Text HLabel 7800 3250 2    50   Input ~ 0
+Text HLabel 7450 3250 2    50   Input ~ 0
 CANL
+$Comp
+L bldc:TJA1051TK-3 U7
+U 1 1 5B1EC10A
+P 5800 3250
+F 0 "U7" H 5725 3715 50  0000 C CNN
+F 1 "TJA1051TK-3" H 5725 3624 50  0000 C CNN
+F 2 "Package_DFN_QFN:DFN-8-1EP_3x3mm_P0.65mm_EP1.55x2.4mm" H 5800 2750 50  0001 C CIN
+F 3 "http://www.nxp.com/documents/data_sheet/TJA1051.pdf" H 5800 3250 50  0001 C CNN
+	1    5800 3250
+	1    0    0    -1
+$EndComp
+Wire Wire Line
+	4950 4000 5700 4000
+Wire Wire Line
+	5700 3550 5700 4000
+Connection ~ 5700 4000
+Wire Wire Line
+	5700 4000 6300 4000
+Wire Wire Line
+	4600 3250 4600 2900
+Connection ~ 4600 3250
+$Comp
+L power:+5V #PWR072
+U 1 1 5B1ECA5A
+P 4600 2900
+F 0 "#PWR072" H 4600 2750 50  0001 C CNN
+F 1 "+5V" H 4615 3073 50  0000 C CNN
+F 2 "" H 4600 2900 50  0001 C CNN
+F 3 "" H 4600 2900 50  0001 C CNN
+	1    4600 2900
+	1    0    0    -1
+$EndComp
+Wire Wire Line
+	6550 3350 6550 2900
+Connection ~ 6550 3350
+$Comp
+L power:VCC #PWR073
+U 1 1 5B1ECE4F
+P 6550 2900
+F 0 "#PWR073" H 6550 2750 50  0001 C CNN
+F 1 "VCC" H 6567 3073 50  0000 C CNN
+F 2 "" H 6550 2900 50  0001 C CNN
+F 3 "" H 6550 2900 50  0001 C CNN
+	1    6550 2900
+	1    0    0    -1
+$EndComp
+Wire Wire Line
+	6550 4000 6550 4150
+Connection ~ 6550 4000
+$Comp
+L power:GND #PWR074
+U 1 1 5B1ED280
+P 6550 4150
+F 0 "#PWR074" H 6550 3900 50  0001 C CNN
+F 1 "GND" H 6555 3977 50  0000 C CNN
+F 2 "" H 6550 4150 50  0001 C CNN
+F 3 "" H 6550 4150 50  0001 C CNN
+	1    6550 4150
+	1    0    0    -1
+$EndComp
 $EndSCHEMATC
