File: design/DRV8301.sch (KiCad schematic (older format))
At the start: 5 parts, among them U2 DRV8302

Commit message: done DRV8301
Parts:
- added C? (x16): C, symbol Device:C
- added D? (x2): LED, symbol Device:LED
- added L?: L, symbol crf_1:L
- added R? (x8): R, symbol Device:R
Connections:
- net labels added: +5V, CS, EN_GATE, FAULT, GH_A, GH_B, GH_C, GL_A, GL_B, GL_C, GND, INH_A, INH_B, INH_C, INL_A, INL_B, INL_C, SCLK, SDI, SDO, SENS_A, SENS_B, SENS_C, SENS_SUPPLY, SH_A, SH_B, SH_C, SL_A, SL_B, SL_C, SUPPLY, VCC
- wire segments 0 -> 106
- no-connect marks 0 -> 5

Commit message: finished schematic and rename LESC to ESCX
Parts:
- added R16: R, symbol Device:R
- gave numbers to parts that had none: 31
Connections:
- wire segments 106 -> 109
- no-connect marks 5 -> 6

Commit message: add value
Parts:
- added C10, C18: 2.2u, symbol Device:C
- added C19: 100u, symbol Device:C
- added L1: 2.2u, symbol Device:L
- added U2: LM3670MF, Package_TO_SOT_SMD:TSOT-23-5, symbol Regulator_Switching:LM3670MF
- C11: renamed from C20; value C -> 2.2u
- C12: renamed from C21; value C -> 2.2u
- C13: renamed from C23; value C -> 2.2u
- C14: renamed from C10; value C -> 6.8n
- C15: renamed from C24; value C -> 2.2u
- C16: renamed from C11; value C -> 120p
- C17: renamed from C18; value C -> 22n
- C20: renamed from C25; value C -> 4.7u_100v
- C21: renamed from C12; value C -> 15n
- C22: renamed from C17; value C -> 220n
- C23: renamed from C19; value C -> 220n
- C24: renamed from C22; value C -> 220n
- C25: renamed from C14; value C -> 100n
- C26: renamed from C13; value C -> 4.7u_100v
- C27: renamed from C15; value C -> 2.2u
- C28: renamed from C16; value C -> 100u
- L2: renamed from L1; value L -> 22u
- R12: value R -> 3.3k
- R13: renamed from R15; value R -> 18k
- R14: value R -> 15k
- R15: renamed from R16; value R -> 10k
- R16: renamed from R13; value R -> 220k
- R17, R19, R21, R23: value R -> 39k
- R18, R20, R22, R24: value R -> 2k2
- renumbered D5 to D4, D4 to D5, U2 to U3
Connections:
- wire segments 109 -> 134

Commit message: add bldc lib, link major component to this lib
Parts:
- removed U3: DRV8302, symbol crf_1:DRV8302
- added U?: DRV8301, symbol bldc:DRV8301
Connections:
- wire segments 134 -> 138
Changed lines of the file:
@@
 $EndDescr
-$Comp
-L crf_1:DRV8302 U3
-U 1 1 5AE19110
-P 5600 2850
-F 0 "U3" H 5600 4487 60  0000 C CNN
-F 1 "DRV8302" H 5600 4381 60  0000 C CNN
-F 2 "" H 5600 2850 60  0001 C CNN
-F 3 "" H 5600 2850 60  0000 C CNN
-	1    5600 2850
-	1    0    0    -1
-$EndComp
 $Comp
 L Device:R R13
@@
 	3200 900  3600 900
 Wire Wire Line
-	3600 1200 3600 1300
+	3600 1200 3600 1250
 Wire Wire Line
 	3600 900  4000 900
@@
 Wire Wire Line
 	4550 1500 4550 1250
-Wire Wire Line
-	3600 1600 3600 1700
-Wire Wire Line
-	3600 1700 4800 1700
-Connection ~ 3600 1600
 NoConn ~ 4800 1800
 NoConn ~ 4800 1900
@@
 	6700 1150 6700 1200
 Wire Wire Line
-	6400 1800 6400 1700
-Wire Wire Line
-	6400 1700 6950 1700
+	6400 1700 6600 1700
 Wire Wire Line
 	6950 1700 6950 1250
@@
 Wire Wire Line
 	7200 1250 7200 1300
-Connection ~ 6400 1700
 Wire Wire Line
 	7200 1250 7350 1250
@@
 SL_C
 Wire Wire Line
-	6400 4100 6400 4000
-Connection ~ 6400 3900
-Wire Wire Line
-	6400 3900 6400 3800
-Connection ~ 6400 4000
-Wire Wire Line
-	6400 4000 6400 3900
-Wire Wire Line
 	6400 3800 6700 3800
-Connection ~ 6400 3800
 $Comp
 L power:GND #PWR045
@@
 	1    0    0    -1
 $EndComp
+Wire Wire Line
+	3600 1250 3850 1250
+Wire Wire Line
+	3850 1250 3850 1700
+Wire Wire Line
+	3850 1700 4800 1700
+Connection ~ 3600 1250
+Wire Wire Line
+	3600 1250 3600 1300
+$Comp
+L bldc:DRV8301 U?
+U 1 1 5B1AF007
+P 5600 2850
+F 0 "U?" H 5600 4487 60  0000 C CNN
+F 1 "DRV8301" H 5600 4381 60  0000 C CNN
+F 2 "" H 5600 2850 60  0000 C CNN
+F 3 "" H 5600 2850 60  0000 C CNN
+	1    5600 2850
+	1    0    0    -1
+$EndComp
+Wire Wire Line
+	6400 1800 6600 1800
+Wire Wire Line
+	6600 1800 6600 1700
+Connection ~ 6600 1700
+Wire Wire Line
+	6600 1700 6950 1700
+Wire Wire Line
+	6400 4100 6400 4000
+Connection ~ 6400 3800
+Connection ~ 6400 3900
+Wire Wire Line
+	6400 3900 6400 3800
+Connection ~ 6400 4000
+Wire Wire Line
+	6400 4000 6400 3900
 $EndSCHEMATC

Commit message: finish sch
Parts:
- removed C19: 100u, symbol Device:C
- removed D4: LED, symbol Device:LED
- removed L2: 22u, symbol crf_1:L
- removed U2: LM3670MF, Package_TO_SOT_SMD:TSOT-23-5, symbol Regulator_Switching:LM3670MF
- added C23: 100u, symbol Device:CP
- added D4: DIODE, symbol Device:D_Schottky
- added L2: 22u, symbol Device:L
- added U2: LM3671, symbol bldc:LM3671
- D5: value LED -> TVS 5V
- U3: renamed from U?; footprint (none) -> Package_SO:HTSSOP-56-1EP_6.1x14mm_P0.5mm_EP3.61x6.35mm
- renumbered C10 to C14, C11 to C15, C12 to C16, C13 to C17, C14 to C18, C15 to C19, C16 to C20, C17 to C21, C18 to C22, C20 to C24, C21 to C25, C22 to C26, C23 to C27, C24 to C28, C25 to C29, C26 to C30, C27 to C31, C28 to C32
