File: design/ESCX.sch (KiCad schematic (older format))
At the start: 22 parts

Commit message: finished schematic and rename LESC to ESCX
Parts:
- added SW1: SENSOR_VOLTAGE, symbol Switch:SW_SPDT
- gave numbers to parts that had none: 22
Connections:
- wire segments 112 -> 111

Commit message: add value
Parts:
- C1: renamed from C2; value C -> 100n
- C2: renamed from C1; value C -> 100n
- R1: renamed from R4; value R -> 2k2
- R10, R11: value R -> 220R
- R2: renamed from R5; value R -> 2k2
- R3: renamed from R6; value R -> 2k2
- R4: renamed from R8; value R -> 100R
- R5: renamed from R1; value R -> 0R
- R6: renamed from R2; value R -> 22R
- R7: renamed from R3; value R -> 22R
- R8: renamed from R7; value R -> 10k
- R9: value R -> 1K
- renumbered J2 to J1, J3 to J2, J4 to J3, J5 to J4, J6 to J5, J1 to J6

Commit message: finish sch
Parts:
- removed J6: USB_OTG, symbol Connector:USB_OTG
- added J6: USB_OTG, symbol bldc:USB_OTG
Changed lines of the file:
@@
 F6 "SCLK" I L 7400 2450 50
 F7 "EN_GATE" I L 7400 2150 50
-F8 "INL_A" I L 7400 1400 50
+F8 "INL_A" I L 7400 1700 50
 F9 "INH_B" I L 7400 1500 50
 F10 "INL_B" I L 7400 1800 50
@@
 F28 "SENS_B" I L 7400 2850 50
 F29 "SENS_C" I L 7400 2950 50
-F30 "INH_A" I L 7400 1700 50
+F30 "INH_A" I L 7400 1400 50
 $EndSheet
 Wire Wire Line
@@
 SUPPLY
 $Comp
-L power:+5V #PWR01
-U 1 1 5AEA140D
-P 1700 7000
-F 0 "#PWR01" H 1700 6850 50  0001 C CNN
-F 1 "+5V" V 1715 7128 50  0000 L CNN
-F 2 "" H 1700 7000 50  0001 C CNN
-F 3 "" H 1700 7000 50  0001 C CNN
-	1    1700 7000
-	0    1    1    0
-$EndComp
-$Comp
 L power:VCC #PWR02
 U 1 1 5AEA14B4
@@
 	1300 7400 1700 7400
 $Comp
-L Connector:USB_OTG J6
-U 1 1 5AEA387A
-P 3050 1400
-F 0 "J6" H 3200 1000 50  0000 C CNN
-F 1 "USB_OTG" V 2800 1300 50  0000 C CNN
-F 2 "" H 3200 1350 50  0001 C CNN
-F 3 " ~" H 3200 1350 50  0001 C CNN
-	1    3050 1400
-	1    0    0    -1
-$EndComp
-$Comp
 L Device:R R6
 U 1 1 5AEA3912
@@
 $EndComp
 $Comp
-L Device:R R5
-U 1 1 5AEA3976
-P 3850 1200
-F 0 "R5" V 3800 1400 50  0000 C CNN
-F 1 "0R" V 3850 1200 50  0000 C CNN
-F 2 "" V 3780 1200 50  0001 C CNN
-F 3 "~" H 3850 1200 50  0001 C CNN
-	1    3850 1200
-	0    1    1    0
-$EndComp
-$Comp
 L power:GND #PWR06
 U 1 1 5AEA3A3B
@@
 Wire Wire Line
 	3350 1400 3700 1400
-Wire Wire Line
-	4150 1200 4150 800
-$Comp
-L power:+5V #PWR018
-U 1 1 5AEA851A
-P 4150 800
-F 0 "#PWR018" H 4150 650 50  0001 C CNN
-F 1 "+5V" H 4165 973 50  0000 C CNN
-F 2 "" H 4150 800 50  0001 C CNN
-F 3 "" H 4150 800 50  0001 C CNN
-	1    4150 800
-	1    0    0    -1
-$EndComp
 $Sheet
 S 3650 2150 600  400
@@
 	0    -1   -1   0
 $EndComp
-Wire Wire Line
-	2950 1800 3050 1800
-Connection ~ 2950 1800
 NoConn ~ 3350 1600
 $Comp
@@
 	1    0    0    -1
 $EndComp
+$Comp
+L bldc:USB_OTG J6
+U 1 1 5B1AFFB0
+P 3050 1400
+F 0 "J6" H 3105 1867 50  0000 C CNN
+F 1 "USB_OTG" H 3105 1776 50  0000 C CNN
+F 2 "" H 3200 1350 50  0001 C CNN
+F 3 " ~" H 3200 1350 50  0001 C CNN
+	1    3050 1400
+	1    0    0    -1
+$EndComp
+Wire Wire Line
+	3050 1800 2950 1800
+Connection ~ 2950 1800
+$Comp
+L Device:R R5
+U 1 1 5B204002
+P 3850 1200
+F 0 "R5" V 3750 1200 50  0000 C CNN
+F 1 "0R" V 3850 1200 50  0000 C CNN
+F 2 "" V 3780 1200 50  0001 C CNN
+F 3 "~" H 3850 1200 50  0001 C CNN
+	1    3850 1200
+	0    1    1    0
+$EndComp
 Wire Wire Line
 	3350 1200 3700 1200
 Wire Wire Line
-	4000 1200 4150 1200
+	4000 1200 4100 1200
+Wire Wire Line
+	4100 1200 4100 850
+$Comp
+L power:+5V #PWR018
+U 1 1 5B20DE34
+P 4100 850
+F 0 "#PWR018" H 4100 700 50  0001 C CNN
+F 1 "+5V" H 4115 1023 50  0000 C CNN
+F 2 "" H 4100 850 50  0001 C CNN
+F 3 "" H 4100 850 50  0001 C CNN
+	1    4100 850
+	1    0    0    -1
+$EndComp
+$Comp
+L power:+5V #PWR01
+U 1 1 5B21418A
+P 1700 7000
+F 0 "#PWR01" H 1700 6850 50  0001 C CNN
+F 1 "+5V" V 1715 7128 50  0000 L CNN
+F 2 "" H 1700 7000 50  0001 C CNN
+F 3 "" H 1700 7000 50  0001 C CNN
+	1    1700 7000
+	0    1    1    0
+$EndComp
 $EndSCHEMATC
