File: design/MPU9150.sch (KiCad schematic (older format))
At the start: 8 parts

Commit message: finished schematic and rename LESC to ESCX
Parts:
- gave numbers to parts that had none: 8
Changed lines of the file:
@@
 EESchema Schematic File Version 4
-LIBS:LESC-cache
+LIBS:ESCX-cache
 EELAYER 26 0
 EELAYER END
@@
 $EndDescr
 $Comp
-L crf_1:MPU9150 U?
+L crf_1:MPU9150 U7
 U 1 1 5AE4C435
 P 5850 3400
-F 0 "U?" H 5825 4415 50  0000 C CNN
+F 0 "U7" H 5825 4415 50  0000 C CNN
 F 1 "MPU9150" H 5825 4324 50  0000 C CNN
 F 2 "" H 5550 3600 50  0001 C CNN
@@
 $EndComp
 $Comp
-L Device:C C?
+L Device:C C43
 U 1 1 5AE4C4B8
 P 4500 2700
-F 0 "C?" V 4248 2700 50  0000 C CNN
+F 0 "C43" V 4248 2700 50  0000 C CNN
 F 1 "C" V 4339 2700 50  0000 C CNN
 F 2 "" H 4538 2550 50  0001 C CNN
@@
 $EndComp
 $Comp
-L Device:C C?
+L Device:C C44
 U 1 1 5AE4C4E7
 P 4500 2950
-F 0 "C?" V 4248 2950 50  0000 C CNN
+F 0 "C44" V 4248 2950 50  0000 C CNN
 F 1 "C" V 4339 2950 50  0000 C CNN
 F 2 "" H 4538 2800 50  0001 C CNN
@@
 $EndComp
 $Comp
-L Device:C C?
+L Device:C C45
 U 1 1 5AE4C51A
 P 6900 3400
-F 0 "C?" H 7015 3446 50  0000 L CNN
+F 0 "C45" H 7015 3446 50  0000 L CNN
 F 1 "C" H 7015 3355 50  0000 L CNN
 F 2 "" H 6938 3250 50  0001 C CNN
@@
 $EndComp
 $Comp
-L Device:C C?
+L Device:C C46
 U 1 1 5AE4C53E
 P 7200 3400
-F 0 "C?" H 7315 3446 50  0000 L CNN
+F 0 "C46" H 7315 3446 50  0000 L CNN
 F 1 "C" H 7315 3355 50  0000 L CNN
 F 2 "" H 7238 3250 50  0001 C CNN
@@
 $EndComp
 $Comp
-L Device:C C?
+L Device:C C47
 U 1 1 5AE4C560
 P 7500 3400
-F 0 "C?" H 7615 3446 50  0000 L CNN
+F 0 "C47" H 7615 3446 50  0000 L CNN
 F 1 "C" H 7615 3355 50  0000 L CNN
 F 2 "" H 7538 3250 50  0001 C CNN
@@
 $EndComp
 $Comp
-L Device:R R?
+L Device:R R40
 U 1 1 5AE4C5F1
 P 4200 3750
-F 0 "R?" H 4270 3796 50  0000 L CNN
+F 0 "R40" H 4270 3796 50  0000 L CNN
 F 1 "R" H 4270 3705 50  0000 L CNN
 F 2 "" V 4130 3750 50  0001 C CNN
@@
 $EndComp
 $Comp
-L Device:R R?
+L Device:R R41
 U 1 1 5AE4C617
 P 4450 3750
-F 0 "R?" H 4520 3796 50  0000 L CNN
+F 0 "R41" H 4520 3796 50  0000 L CNN
 F 1 "R" H 4520 3705 50  0000 L CNN
 F 2 "" V 4380 3750 50  0001 C CNN
@@
 $EndComp
 $Comp
-L power:GND #PWR?
+L power:GND #PWR063
 U 1 1 5AE4C6A6
 P 3900 3100
-F 0 "#PWR?" H 3900 2850 50  0001 C CNN
+F 0 "#PWR063" H 3900 2850 50  0001 C CNN
 F 1 "GND" H 3905 2927 50  0000 C CNN
 F 2 "" H 3900 3100 50  0001 C CNN
@@
 $EndComp
 $Comp
-L power:GND #PWR?
+L power:GND #PWR066
 U 1 1 5AE4C6C8
 P 7500 4250
-F 0 "#PWR?" H 7500 4000 50  0001 C CNN
+F 0 "#PWR066" H 7500 4000 50  0001 C CNN
 F 1 "GND" H 7505 4077 50  0000 C CNN
 F 2 "" H 7500 4250 50  0001 C CNN
@@
 $EndComp
 $Comp
-L power:GND #PWR?
+L power:GND #PWR064
 U 1 1 5AE4C6E3
 P 4750 3400
-F 0 "#PWR?" H 4750 3150 50  0001 C CNN
+F 0 "#PWR064" H 4750 3150 50  0001 C CNN
 F 1 "GND" H 4755 3227 50  0000 C CNN
 F 2 "" H 4750 3400 50  0001 C CNN
@@
 $EndComp
 $Comp
-L power:VCC #PWR?
+L power:VCC #PWR062
 U 1 1 5AE4C763
 P 7500 2550
-F 0 "#PWR?" H 7500 2400 50  0001 C CNN
+F 0 "#PWR062" H 7500 2400 50  0001 C CNN
 F 1 "VCC" H 7517 2723 50  0000 C CNN
 F 2 "" H 7500 2550 50  0001 C CNN
@@
 $EndComp
 $Comp
-L power:VCC #PWR?
+L power:VCC #PWR065
 U 1 1 5AE4C785
 P 4200 3500
-F 0 "#PWR?" H 4200 3350 50  0001 C CNN
+F 0 "#PWR065" H 4200 3350 50  0001 C CNN
 F 1 "VCC" H 4217 3673 50  0000 C CNN
 F 2 "" H 4200 3500 50  0001 C CNN

Commit message: add value
Parts:
- renumbered C43 to C46, C44 to C47, C45 to C48, C46 to C49, C47 to C50, U7 to U8
Changed lines of the file:
@@
 encoding utf-8
 Sheet 6 7
-Title ""
-Date ""
-Rev ""
-Comp ""
+Title "VESC 6.4 redraw"
+Date "2018-06-03"
+Rev "6.4"
+Comp "LI XITONG"
 Comment1 ""
 Comment2 ""
@@
 $EndDescr
 $Comp
-L crf_1:MPU9150 U7
+L crf_1:MPU9150 U8
 U 1 1 5AE4C435
 P 5850 3400
-F 0 "U7" H 5825 4415 50  0000 C CNN
+F 0 "U8" H 5825 4415 50  0000 C CNN
 F 1 "MPU9150" H 5825 4324 50  0000 C CNN
 F 2 "" H 5550 3600 50  0001 C CNN
@@
 $EndComp
 $Comp
-L Device:C C43
+L Device:C C46
 U 1 1 5AE4C4B8
 P 4500 2700
-F 0 "C43" V 4248 2700 50  0000 C CNN
+F 0 "C46" V 4248 2700 50  0000 C CNN
 F 1 "C" V 4339 2700 50  0000 C CNN
 F 2 "" H 4538 2550 50  0001 C CNN
@@
 $EndComp
 $Comp
-L Device:C C44
+L Device:C C47
 U 1 1 5AE4C4E7
 P 4500 2950
-F 0 "C44" V 4248 2950 50  0000 C CNN
+F 0 "C47" V 4248 2950 50  0000 C CNN
 F 1 "C" V 4339 2950 50  0000 C CNN
 F 2 "" H 4538 2800 50  0001 C CNN
@@
 $EndComp
 $Comp
-L Device:C C45
+L Device:C C48
 U 1 1 5AE4C51A
 P 6900 3400
-F 0 "C45" H 7015 3446 50  0000 L CNN
+F 0 "C48" H 7015 3446 50  0000 L CNN
 F 1 "C" H 7015 3355 50  0000 L CNN
 F 2 "" H 6938 3250 50  0001 C CNN
@@
 $EndComp
 $Comp
-L Device:C C46
+L Device:C C49
 U 1 1 5AE4C53E
 P 7200 3400
-F 0 "C46" H 7315 3446 50  0000 L CNN
+F 0 "C49" H 7315 3446 50  0000 L CNN
 F 1 "C" H 7315 3355 50  0000 L CNN
 F 2 "" H 7238 3250 50  0001 C CNN
@@
 $EndComp
 $Comp
-L Device:C C47
+L Device:C C50
 U 1 1 5AE4C560
 P 7500 3400
-F 0 "C47" H 7615 3446 50  0000 L CNN
+F 0 "C50" H 7615 3446 50  0000 L CNN
 F 1 "C" H 7615 3355 50  0000 L CNN
 F 2 "" H 7538 3250 50  0001 C CNN
@@
 $EndComp
 $Comp
-L power:GND #PWR063
+L power:GND #PWR068
 U 1 1 5AE4C6A6
 P 3900 3100
-F 0 "#PWR063" H 3900 2850 50  0001 C CNN
+F 0 "#PWR068" H 3900 2850 50  0001 C CNN
 F 1 "GND" H 3905 2927 50  0000 C CNN
 F 2 "" H 3900 3100 50  0001 C CNN
@@
 $EndComp
 $Comp
-L power:GND #PWR066
+L power:GND #PWR072
 U 1 1 5AE4C6C8
 P 7500 4250
-F 0 "#PWR066" H 7500 4000 50  0001 C CNN
+F 0 "#PWR072" H 7500 4000 50  0001 C CNN
 F 1 "GND" H 7505 4077 50  0000 C CNN
 F 2 "" H 7500 4250 50  0001 C CNN
@@
 $EndComp
 $Comp
-L power:GND #PWR064
+L power:GND #PWR070
 U 1 1 5AE4C6E3
 P 4750 3400
-F 0 "#PWR064" H 4750 3150 50  0001 C CNN
+F 0 "#PWR070" H 4750 3150 50  0001 C CNN
 F 1 "GND" H 4755 3227 50  0000 C CNN
 F 2 "" H 4750 3400 50  0001 C CNN
@@
 $EndComp
 $Comp
-L power:VCC #PWR062
+L power:VCC #PWR071
 U 1 1 5AE4C763
 P 7500 2550
-F 0 "#PWR062" H 7500 2400 50  0001 C CNN
+F 0 "#PWR071" H 7500 2400 50  0001 C CNN
 F 1 "VCC" H 7517 2723 50  0000 C CNN
 F 2 "" H 7500 2550 50  0001 C CNN
@@
 $EndComp
 $Comp
-L power:VCC #PWR065
+L power:VCC #PWR069
 U 1 1 5AE4C785
 P 4200 3500
-F 0 "#PWR065" H 4200 3350 50  0001 C CNN
+F 0 "#PWR069" H 4200 3350 50  0001 C CNN
 F 1 "VCC" H 4217 3673 50  0000 C CNN
 F 2 "" H 4200 3500 50  0001 C CNN

Commit message: finish sch
Parts:
- C50: renamed from C46; value C -> 2.2u
- C51: renamed from C47; value C -> 100n
- C52: renamed from C48; value C -> 2.2u
- C53: renamed from C49; value C -> 2.2u
- C54: renamed from C50; value C -> 2.2u
- R40: value R -> 1K
- R41: value R -> 1k
Changed lines of the file:
@@
 U 1 1 5AE4C435
 P 5850 3400
-F 0 "U8" H 5825 4415 50  0000 C CNN
-F 1 "MPU9150" H 5825 4324 50  0000 C CNN
+F 0 "U8" H 5850 4350 50  0000 C CNN
+F 1 "MPU9150" H 5800 2400 50  0000 C CNN
 F 2 "" H 5550 3600 50  0001 C CNN
 F 3 "" H 5550 3600 50  0001 C CNN
@@
 $EndComp
 $Comp
-L Device:C C46
+L Device:C C50
 U 1 1 5AE4C4B8
 P 4500 2700
-F 0 "C46" V 4248 2700 50  0000 C CNN
-F 1 "C" V 4339 2700 50  0000 C CNN
+F 0 "C50" H 4600 2800 50  0000 C CNN
+F 1 "2.2u" H 4600 2600 50  0000 C CNN
 F 2 "" H 4538 2550 50  0001 C CNN
 F 3 "~" H 4500 2700 50  0001 C CNN
@@
 $EndComp
 $Comp
-L Device:C C47
+L Device:C C51
 U 1 1 5AE4C4E7
 P 4500 2950
-F 0 "C47" V 4248 2950 50  0000 C CNN
-F 1 "C" V 4339 2950 50  0000 C CNN
+F 0 "C51" H 4600 3050 50  0000 C CNN
+F 1 "100n" H 4600 2850 50  0000 C CNN
 F 2 "" H 4538 2800 50  0001 C CNN
 F 3 "~" H 4500 2950 50  0001 C CNN
@@
 $EndComp
 $Comp
-L Device:C C48
+L Device:C C52
 U 1 1 5AE4C51A
 P 6900 3400
-F 0 "C48" H 7015 3446 50  0000 L CNN
-F 1 "C" H 7015 3355 50  0000 L CNN
+F 0 "C52" H 6700 3300 50  0000 L CNN
+F 1 "2.2u" H 6700 3500 50  0000 L CNN
 F 2 "" H 6938 3250 50  0001 C CNN
 F 3 "~" H 6900 3400 50  0001 C CNN
@@
 $EndComp
 $Comp
-L Device:C C49
+L Device:C C53
 U 1 1 5AE4C53E
 P 7200 3400
-F 0 "C49" H 7315 3446 50  0000 L CNN
-F 1 "C" H 7315 3355 50  0000 L CNN
+F 0 "C53" H 7000 3300 50  0000 L CNN
+F 1 "2.2u" H 7000 3500 50  0000 L CNN
 F 2 "" H 7238 3250 50  0001 C CNN
 F 3 "~" H 7200 3400 50  0001 C CNN
@@
 $EndComp
 $Comp
-L Device:C C50
+L Device:C C54
 U 1 1 5AE4C560
 P 7500 3400
-F 0 "C50" H 7615 3446 50  0000 L CNN
-F 1 "C" H 7615 3355 50  0000 L CNN
+F 0 "C54" H 7300 3300 50  0000 L CNN
+F 1 "2.2u" H 7300 3500 50  0000 L CNN
 F 2 "" H 7538 3250 50  0001 C CNN
 F 3 "~" H 7500 3400 50  0001 C CNN
@@
 U 1 1 5AE4C5F1
 P 4200 3750
-F 0 "R40" H 4270 3796 50  0000 L CNN
-F 1 "R" H 4270 3705 50  0000 L CNN
+F 0 "R40" V 4100 3750 50  0000 L CNN
+F 1 "1K" V 4100 3600 50  0000 L CNN
 F 2 "" V 4130 3750 50  0001 C CNN
 F 3 "~" H 4200 3750 50  0001 C CNN
@@
 U 1 1 5AE4C617
 P 4450 3750
-F 0 "R41" H 4520 3796 50  0000 L CNN
-F 1 "R" H 4520 3705 50  0000 L CNN
+F 0 "R41" V 4350 3750 50  0000 L CNN
+F 1 "1k" V 4350 3600 50  0000 L CNN
 F 2 "" V 4380 3750 50  0001 C CNN
 F 3 "~" H 4450 3750 50  0001 C CNN
@@
 $EndComp
 $Comp
-L power:GND #PWR068
+L power:GND #PWR075
 U 1 1 5AE4C6A6
 P 3900 3100
-F 0 "#PWR068" H 3900 2850 50  0001 C CNN
+F 0 "#PWR075" H 3900 2850 50  0001 C CNN
 F 1 "GND" H 3905 2927 50  0000 C CNN
 F 2 "" H 3900 3100 50  0001 C CNN
@@
 $EndComp
 $Comp
-L power:GND #PWR072
+L power:GND #PWR079
 U 1 1 5AE4C6C8
 P 7500 4250
-F 0 "#PWR072" H 7500 4000 50  0001 C CNN
+F 0 "#PWR079" H 7500 4000 50  0001 C CNN
 F 1 "GND" H 7505 4077 50  0000 C CNN
 F 2 "" H 7500 4250 50  0001 C CNN
@@
 $EndComp
 $Comp
-L power:GND #PWR070
+L power:GND #PWR077
 U 1 1 5AE4C6E3
 P 4750 3400
-F 0 "#PWR070" H 4750 3150 50  0001 C CNN
+F 0 "#PWR077" H 4750 3150 50  0001 C CNN
 F 1 "GND" H 4755 3227 50  0000 C CNN
 F 2 "" H 4750 3400 50  0001 C CNN
@@
 $EndComp
 $Comp
-L power:VCC #PWR071
+L power:VCC #PWR078
 U 1 1 5AE4C763
 P 7500 2550
-F 0 "#PWR071" H 7500 2400 50  0001 C CNN
+F 0 "#PWR078" H 7500 2400 50  0001 C CNN
 F 1 "VCC" H 7517 2723 50  0000 C CNN
 F 2 "" H 7500 2550 50  0001 C CNN
@@
 $EndComp
 $Comp
-L power:VCC #PWR069
+L power:VCC #PWR076
 U 1 1 5AE4C785
 P 4200 3500
-F 0 "#PWR069" H 4200 3350 50  0001 C CNN
+F 0 "#PWR076" H 4200 3350 50  0001 C CNN
 F 1 "VCC" H 4217 3673 50  0000 C CNN
 F 2 "" H 4200 3500 50  0001 C CNN
