File: design/NRF.sch (KiCad schematic (older format))
At the start: 1 part

Commit message: finished schematic and rename LESC to ESCX
Parts:
- added C48, C49, C50, C51, C52, C53, C54, C55, C56, C57: C, symbol Device:C
- added L2, L3, L4: INDUCTOR, symbol pspice:INDUCTOR
- added R42: R, symbol Device:R
- added X1: CRYSTAL_GROUND_PIN, symbol crf_1:CRYSTAL_GROUND_PIN
- gave numbers to parts that had none: 1
Connections:
- net labels added: GND, VCC
- wire segments 0 -> 60

Commit message: add value
Parts:
- renumbered C49 to C51, C56 to C52, C48 to C53, C55 to C54, C57 to C55, C50 to C56, C53 to C57, C54 to C58, C51 to C59, C52 to C60, L2 to L4, L4 to L5, U8 to U9
Changed lines of the file:
@@
 encoding utf-8
 Sheet 7 7
-Title ""
-Date ""
-Rev ""
-Comp ""
+Title "VESC 6.4 redraw"
+Date "2018-06-03"
+Rev "6.4"
+Comp "LI XITONG"
 Comment1 ""
 Comment2 ""
@@
 MOSI
 $Comp
-L crf_2:nRF24L01P U8
+L crf_2:nRF24L01P U9
 U 1 1 5AE56EC2
 P 5750 3200
-F 0 "U8" H 6400 3900 50  0000 L CNN
+F 0 "U9" H 6400 3900 50  0000 L CNN
 F 1 "nRF24L01P" H 6250 2550 50  0000 L CNN
 F 2 "Package_DFN_QFN:QFN-20-1EP_4x4mm_P0.5mm_EP2.5x2.5mm" H 5950 4000 50  0001 L CIN
@@
 IRQ
 $Comp
-L Device:C C56
+L Device:C C52
 U 1 1 5AE886AD
 P 5650 4500
-F 0 "C56" H 5765 4546 50  0000 L CNN
+F 0 "C52" H 5765 4546 50  0000 L CNN
 F 1 "C" H 5765 4455 50  0000 L CNN
 F 2 "" H 5688 4350 50  0001 C CNN
@@
 $EndComp
 $Comp
-L Device:C C55
+L Device:C C54
 U 1 1 5AE886CF
 P 6700 4300
-F 0 "C55" V 6448 4300 50  0000 C CNN
+F 0 "C54" V 6448 4300 50  0000 C CNN
 F 1 "C" V 6539 4300 50  0000 C CNN
 F 2 "" H 6738 4150 50  0001 C CNN
@@
 $EndComp
 $Comp
-L Device:C C57
+L Device:C C55
 U 1 1 5AE8871F
 P 6700 4900
-F 0 "C57" V 6448 4900 50  0000 C CNN
+F 0 "C55" V 6448 4900 50  0000 C CNN
 F 1 "C" V 6539 4900 50  0000 C CNN
 F 2 "" H 6738 4750 50  0001 C CNN
@@
 $EndComp
 $Comp
-L power:GND #PWR076
+L power:GND #PWR079
 U 1 1 5AE88987
 P 6850 4900
-F 0 "#PWR076" H 6850 4650 50  0001 C CNN
+F 0 "#PWR079" H 6850 4650 50  0001 C CNN
 F 1 "GND" H 6855 4727 50  0000 C CNN
 F 2 "" H 6850 4900 50  0001 C CNN
@@
 Connection ~ 6550 4300
 $Comp
-L power:GND #PWR074
+L power:GND #PWR076
 U 1 1 5AE88A51
 P 6200 4650
-F 0 "#PWR074" H 6200 4400 50  0001 C CNN
+F 0 "#PWR076" H 6200 4400 50  0001 C CNN
 F 1 "GND" H 6205 4477 50  0000 C CNN
 F 2 "" H 6200 4650 50  0001 C CNN
@@
 $EndComp
 $Comp
-L pspice:INDUCTOR L2
+L pspice:INDUCTOR L4
 U 1 1 5AE8932A
 P 7800 2850
-F 0 "L2" H 7800 2672 50  0000 C CNN
+F 0 "L4" H 7800 2672 50  0000 C CNN
 F 1 "INDUCTOR" H 7800 2763 50  0000 C CNN
 F 2 "" H 7800 2850 50  0001 C CNN
@@
 $EndComp
 $Comp
-L pspice:INDUCTOR L4
+L pspice:INDUCTOR L5
 U 1 1 5AE8937C
 P 7800 3350
-F 0 "L4" H 7800 3172 50  0000 C CNN
+F 0 "L5" H 7800 3172 50  0000 C CNN
 F 1 "INDUCTOR" H 7800 3263 50  0000 C CNN
 F 2 "" H 7800 3350 50  0001 C CNN
@@
 	8200 3350 8050 3350
 $Comp
-L Device:C C53
+L Device:C C57
 U 1 1 5AE89FCA
 P 7550 3700
-F 0 "C53" H 7665 3746 50  0000 L CNN
+F 0 "C57" H 7665 3746 50  0000 L CNN
 F 1 "C" H 7665 3655 50  0000 L CNN
 F 2 "" H 7588 3550 50  0001 C CNN
@@
 	7550 3550 8000 3550
 $Comp
-L Device:C C54
+L Device:C C58
 U 1 1 5AE89FFC
 P 8000 3700
-F 0 "C54" H 8115 3746 50  0000 L CNN
+F 0 "C58" H 8115 3746 50  0000 L CNN
 F 1 "C" H 8115 3655 50  0000 L CNN
 F 2 "" H 8038 3550 50  0001 C CNN
@@
 	8000 3550 8200 3550
 $Comp
-L power:GND #PWR072
+L power:GND #PWR080
 U 1 1 5AE8A097
 P 7550 3850
-F 0 "#PWR072" H 7550 3600 50  0001 C CNN
+F 0 "#PWR080" H 7550 3600 50  0001 C CNN
 F 1 "GND" H 7555 3677 50  0000 C CNN
 F 2 "" H 7550 3850 50  0001 C CNN
@@
 $EndComp
 $Comp
-L power:GND #PWR073
+L power:GND #PWR081
 U 1 1 5AE8A0BD
 P 8000 3850
-F 0 "#PWR073" H 8000 3600 50  0001 C CNN
+F 0 "#PWR081" H 8000 3600 50  0001 C CNN
 F 1 "GND" H 8005 3677 50  0000 C CNN
 F 2 "" H 8000 3850 50  0001 C CNN
@@
 $EndComp
 $Comp
-L Device:C C52
+L Device:C C60
 U 1 1 5AE8A769
 P 8600 3050
-F 0 "C52" H 8715 3096 50  0000 L CNN
+F 0 "C60" H 8715 3096 50  0000 L CNN
 F 1 "C" H 8715 3005 50  0000 L CNN
 F 2 "" H 8638 2900 50  0001 C CNN
@@
 $EndComp
 $Comp
-L Device:C C51
+L Device:C C59
 U 1 1 5AE8A7AF
 P 8350 2850
-F 0 "C51" V 8098 2850 50  0000 C CNN
+F 0 "C59" V 8098 2850 50  0000 C CNN
 F 1 "C" V 8189 2850 50  0000 C CNN
 F 2 "" H 8388 2700 50  0001 C CNN
@@
 $EndComp
 $Comp
-L Device:C C50
+L Device:C C56
 U 1 1 5AE8A9B2
 P 6750 2550
-F 0 "C50" H 6865 2596 50  0000 L CNN
+F 0 "C56" H 6865 2596 50  0000 L CNN
 F 1 "C" H 6865 2505 50  0000 L CNN
 F 2 "" H 6788 2400 50  0001 C CNN
@@
 	6750 2750 6750 2700
 $Comp
-L power:GND #PWR070
+L power:GND #PWR078
 U 1 1 5AE8B277
 P 6850 2800
-F 0 "#PWR070" H 6850 2550 50  0001 C CNN
+F 0 "#PWR078" H 6850 2550 50  0001 C CNN
 F 1 "GND" H 6855 2627 50  0000 C CNN
 F 2 "" H 6850 2800 50  0001 C CNN
@@
 	6750 2300 6750 2400
 $Comp
-L power:VCC #PWR068
+L power:VCC #PWR077
 U 1 1 5AE8BC64
 P 6750 2300
-F 0 "#PWR068" H 6750 2150 50  0001 C CNN
+F 0 "#PWR077" H 6750 2150 50  0001 C CNN
 F 1 "VCC" H 6767 2473 50  0000 C CNN
 F 2 "" H 6750 2300 50  0001 C CNN
@@
 	8600 2850 8600 2900
 $Comp
-L power:GND #PWR071
+L power:GND #PWR082
 U 1 1 5AE8C980
 P 8600 3200
-F 0 "#PWR071" H 8600 2950 50  0001 C CNN
+F 0 "#PWR082" H 8600 2950 50  0001 C CNN
 F 1 "GND" H 8605 3027 50  0000 C CNN
 F 2 "" H 8600 3200 50  0001 C CNN
@@
 Connection ~ 8600 2850
 $Comp
-L Device:C C49
+L Device:C C51
 U 1 1 5AE8D372
 P 5200 2250
-F 0 "C49" H 5315 2296 50  0000 L CNN
+F 0 "C51" H 5315 2296 50  0000 L CNN
 F 1 "C" H 5315 2205 50  0000 L CNN
 F 2 "" H 5238 2100 50  0001 C CNN
@@
 $EndComp
 $Comp
-L Device:C C48
+L Device:C C53
 U 1 1 5AE8D986
 P 5800 2150
-F 0 "C48" H 5915 2196 50  0000 L CNN
+F 0 "C53" H 5915 2196 50  0000 L CNN
 F 1 "C" H 5915 2105 50  0000 L CNN
 F 2 "" H 5838 2000 50  0001 C CNN
@@
 $EndComp
 $Comp
-L power:VCC #PWR067
+L power:VCC #PWR073
 U 1 1 5AE8DAB5
 P 5200 1600
-F 0 "#PWR067" H 5200 1450 50  0001 C CNN
+F 0 "#PWR073" H 5200 1450 50  0001 C CNN
 F 1 "VCC" H 5217 1773 50  0000 C CNN
 F 2 "" H 5200 1600 50  0001 C CNN
@@
 $EndComp
 $Comp
-L power:GND #PWR069
+L power:GND #PWR074
 U 1 1 5AE8DB54
 P 5200 2500
-F 0 "#PWR069" H 5200 2250 50  0001 C CNN
+F 0 "#PWR074" H 5200 2250 50  0001 C CNN
 F 1 "GND" H 5205 2327 50  0000 C CNN
 F 2 "" H 5200 2500 50  0001 C CNN

Commit message: finish sch
Parts:
- C55: renamed from C51; value C -> 100n
- C56: renamed from C52; value C -> 100n
- C57: renamed from C53; value C -> 100n
- C58: renamed from C54; value C -> 15p
- C59: renamed from C55; value C -> 15p
- C60: renamed from C56; value C -> 100n
- C61: renamed from C57; value C -> 2.2n
- C62: renamed from C58; value C -> 4.7p
- C63: renamed from C59; value C -> 1.5p
- C64: renamed from C60; value C -> 1p
- L3: value INDUCTOR -> 8.2n
- L4: value INDUCTOR -> 3.9n
- L5: value INDUCTOR -> 2.7n
- R42: value R -> 22k
- X2: renamed from X1; value CRYSTAL_GROUND_PIN -> 16M
Connections:
- wire segments 60 -> 63
Other:
- note added: "warning! has some error"
Changed lines of the file:
@@
 U 1 1 5AE56EC2
 P 5750 3200
-F 0 "U9" H 6400 3900 50  0000 L CNN
+F 0 "U9" H 6300 3950 50  0000 L CNN
 F 1 "nRF24L01P" H 6250 2550 50  0000 L CNN
 F 2 "Package_DFN_QFN:QFN-20-1EP_4x4mm_P0.5mm_EP2.5x2.5mm" H 5950 4000 50  0001 L CIN
@@
 IRQ
 $Comp
-L Device:C C52
+L Device:C C56
 U 1 1 5AE886AD
 P 5650 4500
-F 0 "C52" H 5765 4546 50  0000 L CNN
-F 1 "C" H 5765 4455 50  0000 L CNN
+F 0 "C56" H 5500 4600 50  0000 L CNN
+F 1 "100n" H 5450 4400 50  0000 L CNN
 F 2 "" H 5688 4350 50  0001 C CNN
 F 3 "~" H 5650 4500 50  0001 C CNN
@@
 $EndComp
 $Comp
-L Device:C C54
+L Device:C C58
 U 1 1 5AE886CF
 P 6700 4300
-F 0 "C54" V 6448 4300 50  0000 C CNN
-F 1 "C" V 6539 4300 50  0000 C CNN
+F 0 "C58" V 6650 4500 50  0000 C CNN
+F 1 "15p" V 6600 4200 50  0000 C CNN
 F 2 "" H 6738 4150 50  0001 C CNN
 F 3 "~" H 6700 4300 50  0001 C CNN
@@
 $EndComp
 $Comp
-L Device:C C55
+L Device:C C59
 U 1 1 5AE8871F
 P 6700 4900
-F 0 "C55" V 6448 4900 50  0000 C CNN
-F 1 "C" V 6539 4900 50  0000 C CNN
+F 0 "C59" V 6600 5150 50  0000 C CNN
+F 1 "15p" V 6550 4850 50  0000 C CNN
 F 2 "" H 6738 4750 50  0001 C CNN
 F 3 "~" H 6700 4900 50  0001 C CNN
@@
 $EndComp
 $Comp
-L crf_1:CRYSTAL_GROUND_PIN X1
+L crf_1:CRYSTAL_GROUND_PIN X2
 U 1 1 5AE887EC
 P 6550 4600
-F 0 "X1" V 6497 4733 60  0000 L CNN
-F 1 "CRYSTAL_GROUND_PIN" V 6603 4733 60  0000 L CNN
-F 2 "" H 6550 4600 60  0000 C CNN
+F 0 "X2" V 6500 4700 60  0000 L CNN
+F 1 "16M" V 6600 4700 60  0000 L CNN
+F 2 "" H 6550 4600 60  0001 C CNN
 F 3 "" H 6550 4600 60  0000 C CNN
 	1    6550 4600
@@
 $EndComp
 $Comp
-L power:GND #PWR079
+L power:GND #PWR087
 U 1 1 5AE88987
 P 6850 4900
-F 0 "#PWR079" H 6850 4650 50  0001 C CNN
+F 0 "#PWR087" H 6850 4650 50  0001 C CNN
 F 1 "GND" H 6855 4727 50  0000 C CNN
 F 2 "" H 6850 4900 50  0001 C CNN
@@
 $EndComp
 $Comp
-L power:GND #PWR075
+L power:GND #PWR083
 U 1 1 5AE889A3
 P 5650 4850
-F 0 "#PWR075" H 5650 4600 50  0001 C CNN
+F 0 "#PWR083" H 5650 4600 50  0001 C CNN
 F 1 "GND" H 5655 4677 50  0000 C CNN
 F 2 "" H 5650 4850 50  0001 C CNN
@@
 $EndComp
 Wire Wire Line
-	5650 3900 5650 4350
+	5650 3900 5650 4200
 Wire Wire Line
 	5650 4650 5650 4800
@@
 Connection ~ 6550 4300
 $Comp
-L power:GND #PWR076
+L power:GND #PWR084
 U 1 1 5AE88A51
 P 6200 4650
-F 0 "#PWR076" H 6200 4400 50  0001 C CNN
+F 0 "#PWR084" H 6200 4400 50  0001 C CNN
 F 1 "GND" H 6205 4477 50  0000 C CNN
 F 2 "" H 6200 4650 50  0001 C CNN
@@
 P 7150 3100
 F 0 "L3" V 7104 3178 50  0000 L CNN
-F 1 "INDUCTOR" V 7195 3178 50  0000 L CNN
+F 1 "8.2n" V 7195 3178 50  0000 L CNN
 F 2 "" H 7150 3100 50  0001 C CNN
 F 3 "" H 7150 3100 50  0001 C CNN
@@
 P 7800 2850
 F 0 "L4" H 7800 2672 50  0000 C CNN
-F 1 "INDUCTOR" H 7800 2763 50  0000 C CNN
+F 1 "3.9n" H 7800 2763 50  0000 C CNN
 F 2 "" H 7800 2850 50  0001 C CNN
 F 3 "" H 7800 2850 50  0001 C CNN
@@
 P 7800 3350
 F 0 "L5" H 7800 3172 50  0000 C CNN
-F 1 "INDUCTOR" H 7800 3263 50  0000 C CNN
+F 1 "2.7n" H 7800 3263 50  0000 C CNN
 F 2 "" H 7800 3350 50  0001 C CNN
 F 3 "" H 7800 3350 50  0001 C CNN
@@
 	8200 3350 8050 3350
 $Comp
-L Device:C C57
+L Device:C C61
 U 1 1 5AE89FCA
 P 7550 3700
-F 0 "C57" H 7665 3746 50  0000 L CNN
-F 1 "C" H 7665 3655 50  0000 L CNN
+F 0 "C61" H 7665 3746 50  0000 L CNN
+F 1 "2.2n" H 7665 3655 50  0000 L CNN
 F 2 "" H 7588 3550 50  0001 C CNN
 F 3 "~" H 7550 3700 50  0001 C CNN
@@
 	7550 3550 8000 3550
 $Comp
-L Device:C C58
+L Device:C C62
 U 1 1 5AE89FFC
 P 8000 3700
-F 0 "C58" H 8115 3746 50  0000 L CNN
-F 1 "C" H 8115 3655 50  0000 L CNN
+F 0 "C62" H 8115 3746 50  0000 L CNN
+F 1 "4.7p" H 8115 3655 50  0000 L CNN
 F 2 "" H 8038 3550 50  0001 C CNN
 F 3 "~" H 8000 3700 50  0001 C CNN
@@
 	8000 3550 8200 3550
 $Comp
-L power:GND #PWR080
+L power:GND #PWR088
 U 1 1 5AE8A097
 P 7550 3850
-F 0 "#PWR080" H 7550 3600 50  0001 C CNN
+F 0 "#PWR088" H 7550 3600 50  0001 C CNN
 F 1 "GND" H 7555 3677 50  0000 C CNN
 F 2 "" H 7550 3850 50  0001 C CNN
@@
 $EndComp
 $Comp
-L power:GND #PWR081
+L power:GND #PWR089
 U 1 1 5AE8A0BD
 P 8000 3850
-F 0 "#PWR081" H 8000 3600 50  0001 C CNN
+F 0 "#PWR089" H 8000 3600 50  0001 C CNN
 F 1 "GND" H 8005 3677 50  0000 C CNN
 F 2 "" H 8000 3850 50  0001 C CNN
@@
 $EndComp
 $Comp
-L Device:C C60
+L Device:C C64
 U 1 1 5AE8A769
 P 8600 3050
-F 0 "C60" H 8715 3096 50  0000 L CNN
-F 1 "C" H 8715 3005 50  0000 L CNN
+F 0 "C64" H 8715 3096 50  0000 L CNN
+F 1 "1p" H 8715 3005 50  0000 L CNN
 F 2 "" H 8638 2900 50  0001 C CNN
 F 3 "~" H 8600 3050 50  0001 C CNN
@@
 $EndComp
 $Comp
-L Device:C C59
+L Device:C C63
 U 1 1 5AE8A7AF
 P 8350 2850
-F 0 "C59" V 8098 2850 50  0000 C CNN
-F 1 "C" V 8189 2850 50  0000 C CNN
+F 0 "C63" V 8098 2850 50  0000 C CNN
+F 1 "1.5p" V 8189 2850 50  0000 C CNN
 F 2 "" H 8388 2700 50  0001 C CNN
 F 3 "~" H 8350 2850 50  0001 C CNN
@@
 $EndComp
 $Comp
-L Device:C C56
+L Device:C C60
 U 1 1 5AE8A9B2
 P 6750 2550
-F 0 "C56" H 6865 2596 50  0000 L CNN
-F 1 "C" H 6865 2505 50  0000 L CNN
+F 0 "C60" H 6865 2596 50  0000 L CNN
+F 1 "100n" H 6865 2505 50  0000 L CNN
 F 2 "" H 6788 2400 50  0001 C CNN
 F 3 "~" H 6750 2550 50  0001 C CNN
@@
 	6750 2750 6750 2700
 $Comp
-L power:GND #PWR078
+L power:GND #PWR086
 U 1 1 5AE8B277
 P 6850 2800
-F 0 "#PWR078" H 6850 2550 50  0001 C CNN
+F 0 "#PWR086" H 6850 2550 50  0001 C CNN
 F 1 "GND" H 6855 2627 50  0000 C CNN
 F 2 "" H 6850 2800 50  0001 C CNN
@@
 	6750 2300 6750 2400
 $Comp
-L power:VCC #PWR077
+L power:VCC #PWR085
 U 1 1 5AE8BC64
 P 6750 2300
-F 0 "#PWR077" H 6750 2150 50  0001 C CNN
+F 0 "#PWR085" H 6750 2150 50  0001 C CNN
 F 1 "VCC" H 6767 2473 50  0000 C CNN
 F 2 "" H 6750 2300 50  0001 C CNN
@@
 	8600 2850 8600 2900
 $Comp
-L power:GND #PWR082
+L power:GND #PWR090
 U 1 1 5AE8C980
 P 8600 3200
-F 0 "#PWR082" H 8600 2950 50  0001 C CNN
+F 0 "#PWR090" H 8600 2950 50  0001 C CNN
 F 1 "GND" H 8605 3027 50  0000 C CNN
 F 2 "" H 8600 3200 50  0001 C CNN
@@
 Connection ~ 8600 2850
 $Comp
-L Device:C C51
+L Device:C C55
 U 1 1 5AE8D372
 P 5200 2250
-F 0 "C51" H 5315 2296 50  0000 L CNN
-F 1 "C" H 5315 2205 50  0000 L CNN
+F 0 "C55" H 5250 2350 50  0000 L CNN
+F 1 "100n" H 5250 2150 50  0000 L CNN
 F 2 "" H 5238 2100 50  0001 C CNN
 F 3 "~" H 5200 2250 50  0001 C CNN
@@
 $EndComp
 $Comp
-L Device:C C53
+L Device:C C57
 U 1 1 5AE8D986
 P 5800 2150
-F 0 "C53" H 5915 2196 50  0000 L CNN
-F 1 "C" H 5915 2105 50  0000 L CNN
+F 0 "C57" V 5850 2200 50  0000 L CNN
+F 1 "100n" V 5850 1900 50  0000 L CNN
 F 2 "" H 5838 2000 50  0001 C CNN
 F 3 "~" H 5800 2150 50  0001 C CNN
@@
 P 6100 2150
 F 0 "R42" H 6170 2196 50  0000 L CNN
-F 1 "R" H 6170 2105 50  0000 L CNN
+F 1 "22k" H 6170 2105 50  0000 L CNN
 F 2 "" V 6030 2150 50  0001 C CNN
 F 3 "~" H 6100 2150 50  0001 C CNN
@@
 $EndComp
 $Comp
-L power:VCC #PWR073
+L power:VCC #PWR080
 U 1 1 5AE8DAB5
 P 5200 1600
-F 0 "#PWR073" H 5200 1450 50  0001 C CNN
+F 0 "#PWR080" H 5200 1450 50  0001 C CNN
 F 1 "VCC" H 5217 1773 50  0000 C CNN
 F 2 "" H 5200 1600 50  0001 C CNN
@@
 $EndComp
 $Comp
-L power:GND #PWR074
+L power:GND #PWR081
 U 1 1 5AE8DB54
 P 5200 2500
-F 0 "#PWR074" H 5200 2250 50  0001 C CNN
+F 0 "#PWR081" H 5200 2250 50  0001 C CNN
 F 1 "GND" H 5205 2327 50  0000 C CNN
 F 2 "" H 5200 2500 50  0001 C CNN
@@
 	5200 2450 5200 2500
 Connection ~ 5600 1850
+$Comp
+L power:GND #PWR091
+U 1 1 5B1F54BB
+P 9350 3100
+F 0 "#PWR091" H 9350 2850 50  0001 C CNN
+F 1 "GND" H 9355 2927 50  0000 C CNN
+F 2 "" H 9350 3100 50  0001 C CNN
+F 3 "" H 9350 3100 50  0001 C CNN
+	1    9350 3100
+	1    0    0    -1
+$EndComp
+Wire Wire Line
+	5650 4200 5200 4200
+Wire Wire Line
+	5200 4200 5200 4150
+Connection ~ 5650 4200
+Wire Wire Line
+	5650 4200 5650 4350
+$Comp
+L power:VCC #PWR082
+U 1 1 5B1F676F
+P 5200 4150
+F 0 "#PWR082" H 5200 4000 50  0001 C CNN
+F 1 "VCC" H 5217 4323 50  0000 C CNN
+F 2 "" H 5200 4150 50  0001 C CNN
+F 3 "" H 5200 4150 50  0001 C CNN
+	1    5200 4150
+	1    0    0    -1
+$EndComp
+Text Notes 9200 3450 0    50   ~ 0
+warning! has some error
 $EndSCHEMATC
