File: design/mcu.sch (KiCad schematic (older format))
At the start: 9 parts, among them U1 STM32F40X_LQFP64, Y1 Crystal

Commit message: finished schematic and rename LESC to ESCX
Parts:
- renumbered C1 to C3, C6 to C4, C4 to C5, C5 to C6, C2 to C8, C3 to C9
Changed lines of the file:
@@
 EESchema Schematic File Version 4
-LIBS:LESC-cache
+LIBS:ESCX-cache
 EELAYER 26 0
 EELAYER END
@@
 NoConn ~ 6600 1250
 $Comp
-L Device:C C1
+L Device:C C3
 U 1 1 5AE152D5
 P 7000 1250
-F 0 "C1" H 7115 1296 50  0000 L CNN
+F 0 "C3" H 7115 1296 50  0000 L CNN
 F 1 "C" H 7115 1205 50  0000 L CNN
 F 2 "" H 7038 1100 50  0001 C CNN
@@
 $EndComp
 $Comp
-L Device:C C6
+L Device:C C4
 U 1 1 5AE1530D
 P 7500 1250
-F 0 "C6" H 7615 1296 50  0000 L CNN
+F 0 "C4" H 7615 1296 50  0000 L CNN
 F 1 "C" H 7615 1205 50  0000 L CNN
 F 2 "" H 7538 1100 50  0001 C CNN
@@
 Connection ~ 7500 1100
 $Comp
-L power:GND #PWR0101
+L power:GND #PWR022
 U 1 1 5AE15823
 P 7850 1150
-F 0 "#PWR0101" H 7850 900 50  0001 C CNN
+F 0 "#PWR022" H 7850 900 50  0001 C CNN
 F 1 "GND" H 7855 977 50  0000 C CNN
 F 2 "" H 7850 1150 50  0001 C CNN
@@
 $EndComp
 $Comp
-L power:GND #PWR0102
+L power:GND #PWR023
 U 1 1 5AE159D5
 P 6900 1750
-F 0 "#PWR0102" H 6900 1500 50  0001 C CNN
+F 0 "#PWR023" H 6900 1500 50  0001 C CNN
 F 1 "GND" H 6905 1577 50  0000 C CNN
 F 2 "" H 6900 1750 50  0001 C CNN
@@
 NRST
 $Comp
-L Device:C C4
+L Device:C C5
 U 1 1 5AE15FB9
 P 7150 2300
-F 0 "C4" H 7265 2346 50  0000 L CNN
+F 0 "C5" H 7265 2346 50  0000 L CNN
 F 1 "C" H 7265 2255 50  0000 L CNN
 F 2 "" H 7188 2150 50  0001 C CNN
@@
 $EndComp
 $Comp
-L power:GND #PWR0103
+L power:GND #PWR024
 U 1 1 5AE16023
 P 7150 2450
-F 0 "#PWR0103" H 7150 2200 50  0001 C CNN
+F 0 "#PWR024" H 7150 2200 50  0001 C CNN
 F 1 "GND" H 7155 2277 50  0000 C CNN
 F 2 "" H 7150 2450 50  0001 C CNN
@@
 PB4
 $Comp
-L power:VCC #PWR0104
+L power:VCC #PWR025
 U 1 1 5AE16835
 P 6600 3500
-F 0 "#PWR0104" H 6600 3350 50  0001 C CNN
+F 0 "#PWR025" H 6600 3350 50  0001 C CNN
 F 1 "VCC" H 6617 3673 50  0000 C CNN
 F 2 "" H 6600 3500 50  0001 C CNN
@@
 	6600 3950 6600 4050
 $Comp
-L power:GND #PWR0105
+L power:GND #PWR026
 U 1 1 5AE16A27
 P 6600 4450
-F 0 "#PWR0105" H 6600 4200 50  0001 C CNN
+F 0 "#PWR026" H 6600 4200 50  0001 C CNN
 F 1 "GND" H 6605 4277 50  0000 C CNN
 F 2 "" H 6600 4450 50  0001 C CNN
@@
 Connection ~ 6600 4450
 $Comp
-L power:VCC #PWR0106
+L power:VCC #PWR027
 U 1 1 5AE16BF8
 P 6600 4850
-F 0 "#PWR0106" H 6600 4700 50  0001 C CNN
+F 0 "#PWR027" H 6600 4700 50  0001 C CNN
 F 1 "VCC" H 6617 5023 50  0000 C CNN
 F 2 "" H 6600 4850 50  0001 C CNN
@@
 $EndComp
 $Comp
-L power:VCC #PWR0107
+L power:VCC #PWR028
 U 1 1 5AE16C41
 P 7000 4850
-F 0 "#PWR0107" H 7000 4700 50  0001 C CNN
+F 0 "#PWR028" H 7000 4700 50  0001 C CNN
 F 1 "VCC" H 7017 5023 50  0000 C CNN
 F 2 "" H 7000 4850 50  0001 C CNN
@@
 $EndComp
 $Comp
-L Device:C C5
+L Device:C C6
 U 1 1 5AE16C87
 P 7250 5000
-F 0 "C5" H 7365 5046 50  0000 L CNN
+F 0 "C6" H 7365 5046 50  0000 L CNN
 F 1 "C" H 7365 4955 50  0000 L CNN
 F 2 "" H 7288 4850 50  0001 C CNN
@@
 Connection ~ 7600 5150
 $Comp
-L power:GND #PWR0108
+L power:GND #PWR029
 U 1 1 5AE1756F
 P 7600 5300
-F 0 "#PWR0108" H 7600 5050 50  0001 C CNN
+F 0 "#PWR029" H 7600 5050 50  0001 C CNN
 F 1 "GND" H 7605 5127 50  0000 C CNN
 F 2 "" H 7600 5300 50  0001 C CNN
@@
 $EndComp
 $Comp
-L Device:C C2
+L Device:C C8
 U 1 1 5AE175BB
 P 7100 5400
-F 0 "C2" V 7050 5300 50  0000 C CNN
+F 0 "C8" V 7050 5300 50  0000 C CNN
 F 1 "C" V 6939 5400 50  0000 C CNN
 F 2 "" H 7138 5250 50  0001 C CNN
@@
 $EndComp
 $Comp
-L Device:C C3
+L Device:C C9
 U 1 1 5AE175F4
 P 7100 5650
-F 0 "C3" V 7200 5550 50  0000 C CNN
+F 0 "C9" V 7200 5550 50  0000 C CNN
 F 1 "C" V 7250 5650 50  0000 C CNN
 F 2 "" H 7138 5500 50  0001 C CNN

Commit message: add value
Parts:
- C3: value C -> 15p
- C4: renamed from C8; value C -> 2.2u
- C5: renamed from C9; value C -> 2.2u
- C6: renamed from C5; value C -> 100n
- C7: renamed from C6; value C -> 2.2u
- C8: renamed from C4; value C -> 15p
- C9: renamed from C7; value C -> 2.2u
- Y1: value Crystal -> 8m
Changed lines of the file:
@@
 Sheet 2 7
 Title "VESC 6.4 redraw"
-Date "2018-04-26"
+Date "2018-06-03"
 Rev "6.4"
 Comp "LI XITONG"
@@
 U 1 1 5AE152D5
 P 7000 1250
-F 0 "C3" H 7115 1296 50  0000 L CNN
-F 1 "C" H 7115 1205 50  0000 L CNN
+F 0 "C3" H 7000 1350 50  0000 L CNN
+F 1 "15p" H 7000 1150 50  0000 L CNN
 F 2 "" H 7038 1100 50  0001 C CNN
 F 3 "~" H 7000 1250 50  0001 C CNN
@@
 $EndComp
 $Comp
-L Device:C C4
+L Device:C C8
 U 1 1 5AE1530D
 P 7500 1250
-F 0 "C4" H 7615 1296 50  0000 L CNN
-F 1 "C" H 7615 1205 50  0000 L CNN
+F 0 "C8" H 7550 1350 50  0000 L CNN
+F 1 "15p" H 7550 1150 50  0000 L CNN
 F 2 "" H 7538 1100 50  0001 C CNN
 F 3 "~" H 7500 1250 50  0001 C CNN
@@
 U 1 1 5AE15619
 P 7250 1400
-F 0 "Y1" H 7250 1668 50  0000 C CNN
-F 1 "Crystal" H 7250 1577 50  0000 C CNN
+F 0 "Y1" H 7250 1550 50  0000 C CNN
+F 1 "8m" H 7400 1300 50  0000 C CNN
 F 2 "" H 7250 1400 50  0001 C CNN
 F 3 "~" H 7250 1400 50  0001 C CNN
@@
 Connection ~ 7500 1100
 $Comp
-L power:GND #PWR022
+L power:GND #PWR031
 U 1 1 5AE15823
 P 7850 1150
-F 0 "#PWR022" H 7850 900 50  0001 C CNN
+F 0 "#PWR031" H 7850 900 50  0001 C CNN
 F 1 "GND" H 7855 977 50  0000 C CNN
 F 2 "" H 7850 1150 50  0001 C CNN
@@
 $EndComp
 $Comp
-L power:GND #PWR023
+L power:GND #PWR027
 U 1 1 5AE159D5
 P 6900 1750
-F 0 "#PWR023" H 6900 1500 50  0001 C CNN
+F 0 "#PWR027" H 6900 1500 50  0001 C CNN
 F 1 "GND" H 6905 1577 50  0000 C CNN
 F 2 "" H 6900 1750 50  0001 C CNN
@@
 NRST
 $Comp
-L Device:C C5
+L Device:C C6
 U 1 1 5AE15FB9
 P 7150 2300
-F 0 "C5" H 7265 2346 50  0000 L CNN
-F 1 "C" H 7265 2255 50  0000 L CNN
+F 0 "C6" H 7265 2346 50  0000 L CNN
+F 1 "100n" H 7250 2200 50  0000 L CNN
 F 2 "" H 7188 2150 50  0001 C CNN
 F 3 "~" H 7150 2300 50  0001 C CNN
@@
 $EndComp
 $Comp
-L power:GND #PWR024
+L power:GND #PWR029
 U 1 1 5AE16023
 P 7150 2450
-F 0 "#PWR024" H 7150 2200 50  0001 C CNN
+F 0 "#PWR029" H 7150 2200 50  0001 C CNN
 F 1 "GND" H 7155 2277 50  0000 C CNN
 F 2 "" H 7150 2450 50  0001 C CNN
@@
 PB4
 $Comp
-L power:VCC #PWR025
+L power:VCC #PWR024
 U 1 1 5AE16835
 P 6600 3500
-F 0 "#PWR025" H 6600 3350 50  0001 C CNN
+F 0 "#PWR024" H 6600 3350 50  0001 C CNN
 F 1 "VCC" H 6617 3673 50  0000 C CNN
 F 2 "" H 6600 3500 50  0001 C CNN
@@
 	6600 3950 6600 4050
 $Comp
-L power:GND #PWR026
+L power:GND #PWR025
 U 1 1 5AE16A27
 P 6600 4450
-F 0 "#PWR026" H 6600 4200 50  0001 C CNN
-F 1 "GND" H 6605 4277 50  0000 C CNN
+F 0 "#PWR025" H 6600 4200 50  0001 C CNN
+F 1 "GND" H 6700 4350 50  0000 C CNN
 F 2 "" H 6600 4450 50  0001 C CNN
 F 3 "" H 6600 4450 50  0001 C CNN
@@
 Connection ~ 6600 4450
 $Comp
-L power:VCC #PWR027
+L power:VCC #PWR026
 U 1 1 5AE16BF8
 P 6600 4850
-F 0 "#PWR027" H 6600 4700 50  0001 C CNN
-F 1 "VCC" H 6617 5023 50  0000 C CNN
+F 0 "#PWR026" H 6600 4700 50  0001 C CNN
+F 1 "VCC" H 6700 4950 50  0000 C CNN
 F 2 "" H 6600 4850 50  0001 C CNN
 F 3 "" H 6600 4850 50  0001 C CNN
@@
 P 7000 4850
 F 0 "#PWR028" H 7000 4700 50  0001 C CNN
-F 1 "VCC" H 7017 5023 50  0000 C CNN
+F 1 "VCC" H 7000 5000 50  0000 C CNN
 F 2 "" H 7000 4850 50  0001 C CNN
 F 3 "" H 7000 4850 50  0001 C CNN
@@
 $EndComp
 $Comp
-L Device:C C6
+L Device:C C7
 U 1 1 5AE16C87
 P 7250 5000
-F 0 "C6" H 7365 5046 50  0000 L CNN
-F 1 "C" H 7365 4955 50  0000 L CNN
+F 0 "C7" H 7350 5100 50  0000 L CNN
+F 1 "2.2u" H 7350 5000 50  0000 L CNN
 F 2 "" H 7288 4850 50  0001 C CNN
 F 3 "~" H 7250 5000 50  0001 C CNN
@@
 $EndComp
 $Comp
-L Device:C C7
+L Device:C C9
 U 1 1 5AE16CBF
 P 7600 5000
-F 0 "C7" H 7715 5046 50  0000 L CNN
-F 1 "C" H 7715 4955 50  0000 L CNN
+F 0 "C9" H 7700 5100 50  0000 L CNN
+F 1 "2.2u" H 7700 5000 50  0000 L CNN
 F 2 "" H 7638 4850 50  0001 C CNN
 F 3 "~" H 7600 5000 50  0001 C CNN
@@
 Connection ~ 7600 5150
 $Comp
-L power:GND #PWR029
+L power:GND #PWR030
 U 1 1 5AE1756F
 P 7600 5300
-F 0 "#PWR029" H 7600 5050 50  0001 C CNN
+F 0 "#PWR030" H 7600 5050 50  0001 C CNN
 F 1 "GND" H 7605 5127 50  0000 C CNN
 F 2 "" H 7600 5300 50  0001 C CNN
@@
 $EndComp
 $Comp
-L Device:C C8
+L Device:C C4
 U 1 1 5AE175BB
 P 7100 5400
-F 0 "C8" V 7050 5300 50  0000 C CNN
-F 1 "C" V 6939 5400 50  0000 C CNN
+F 0 "C4" V 7150 5500 50  0000 C CNN
+F 1 "2.2u" H 7200 5300 50  0000 C CNN
 F 2 "" H 7138 5250 50  0001 C CNN
 F 3 "~" H 7100 5400 50  0001 C CNN
@@
 $EndComp
 $Comp
-L Device:C C9
+L Device:C C5
 U 1 1 5AE175F4
 P 7100 5650
-F 0 "C9" V 7200 5550 50  0000 C CNN
-F 1 "C" V 7250 5650 50  0000 C CNN
+F 0 "C5" V 7200 5750 50  0000 C CNN
+F 1 "2.2u" H 7200 5550 50  0000 C CNN
 F 2 "" H 7138 5500 50  0001 C CNN
 F 3 "~" H 7100 5650 50  0001 C CNN

Commit message: add bldc lib, link major component to this lib
Parts:
- removed U1: STM32F40X_LQFP64, symbol crf_1:STM32F40X_LQFP64
- added U?: STM32F40X_LQFP64, symbol bldc:STM32F40X_LQFP64
Changed lines of the file:
@@
 Comment4 ""
 $EndDescr
-$Comp
-L crf_1:STM32F40X_LQFP64 U1
-U 1 1 5AE14E6D
-P 5350 3300
-F 0 "U1" H 5350 5737 60  0000 C CNN
-F 1 "STM32F40X_LQFP64" H 5350 5631 60  0000 C CNN
-F 2 "" H 5350 3300 60  0001 C CNN
-F 3 "" H 5350 3300 60  0000 C CNN
-	1    5350 3300
-	1    0    0    -1
-$EndComp
 Text HLabel 4100 1150 0    50   Input ~ 0
 VOLTAGE_1
@@
 	1    0    0    -1
 $EndComp
-Wire Wire Line
-	6600 3500 6600 3750
-Connection ~ 6600 3750
-Wire Wire Line
-	6600 3750 6600 3850
-Connection ~ 6600 3850
-Wire Wire Line
-	6600 3850 6600 3950
-Connection ~ 6600 3950
-Wire Wire Line
-	6600 3950 6600 4050
 $Comp
 L power:GND #PWR025
@@
 	1    0    0    -1
 $EndComp
-Wire Wire Line
-	6600 4350 6600 4450
-Connection ~ 6600 4450
 $Comp
 L power:VCC #PWR026
@@
 Wire Wire Line
 	6750 5650 6950 5650
+Wire Wire Line
+	6600 3500 6600 3750
+$Comp
+L bldc:STM32F40X_LQFP64 U?
+U 1 1 5B1B9E2F
+P 5350 3300
+F 0 "U?" H 5350 5737 60  0000 C CNN
+F 1 "STM32F40X_LQFP64" H 5350 5631 60  0000 C CNN
+F 2 "" H 5350 3300 60  0000 C CNN
+F 3 "" H 5350 3300 60  0000 C CNN
+	1    5350 3300
+	1    0    0    -1
+$EndComp
+Wire Wire Line
+	6600 4050 6600 3950
+Connection ~ 6600 3750
+Connection ~ 6600 3850
+Wire Wire Line
+	6600 3850 6600 3750
+Connection ~ 6600 3950
+Wire Wire Line
+	6600 3950 6600 3850
+Wire Wire Line
+	6600 4350 6600 4450
+Connection ~ 6600 4450
 $EndSCHEMATC

Commit message: finish sch
Parts:
- removed Y1: 8m, symbol Device:Crystal
- added C10, C11, C12, C13: 2.2u, symbol Device:C
- added X1: 8m, symbol crf_1:CRYSTAL_GROUND_PIN
- U1: renamed from U?; footprint (none) -> Package_QFP:LQFP-64_10x10mm_P0.5mm
- renumbered C9 to C8, C8 to C9
Connections:
- wire segments 33 -> 41
Other:
- note added: "Bypass, place next to VDD pins"
