File: design/power.sch (KiCad schematic (older format))
At the start: 0 parts

Commit message: done DRV8301
Parts:
- added Q? (x6): IRF7748L1, Package_DirectFET:DirectFET_L6, symbol Transistor_FET:IRF7748L1
- added U? (x3): AD8418, symbol Amplifier_Current:AD8418
Changed lines of the file:
@@
 Comment4 ""
 $EndDescr
+$Comp
+L Amplifier_Current:AD8418 U?
+U 1 1 5AE64709
+P 1950 2800
+F 0 "U?" H 1950 2314 50  0000 C CNN
+F 1 "AD8418" H 1950 2223 50  0000 C CNN
+F 2 "" H 2000 2450 50  0001 C CNN
+F 3 "http://www.analog.com/media/en/technical-documentation/data-sheets/AD8418.pdf" H 2600 2100 50  0001 C CNN
+	1    1950 2800
+	1    0    0    -1
+$EndComp
+$Comp
+L Amplifier_Current:AD8418 U?
+U 1 1 5AE6479F
+P 5250 2850
+F 0 "U?" H 5250 2364 50  0000 C CNN
+F 1 "AD8418" H 5250 2273 50  0000 C CNN
+F 2 "" H 5300 2500 50  0001 C CNN
+F 3 "http://www.analog.com/media/en/technical-documentation/data-sheets/AD8418.pdf" H 5900 2150 50  0001 C CNN
+	1    5250 2850
+	1    0    0    -1
+$EndComp
+$Comp
+L Amplifier_Current:AD8418 U?
+U 1 1 5AE6486D
+P 8300 2850
+F 0 "U?" H 8300 2364 50  0000 C CNN
+F 1 "AD8418" H 8300 2273 50  0000 C CNN
+F 2 "" H 8350 2500 50  0001 C CNN
+F 3 "http://www.analog.com/media/en/technical-documentation/data-sheets/AD8418.pdf" H 8950 2150 50  0001 C CNN
+	1    8300 2850
+	1    0    0    -1
+$EndComp
+$Comp
+L Transistor_FET:IRF7748L1 Q?
+U 1 1 5AE649B5
+P 3450 1550
+F 0 "Q?" H 3656 1596 50  0000 L CNN
+F 1 "IRF7748L1" H 3656 1505 50  0000 L CNN
+F 2 "Package_DirectFET:DirectFET_L6" H 3450 1550 50  0001 C CIN
+F 3 "https://www.infineon.com/dgdl/irf7748l1pbf.pdf?fileId=5546d462533600a40153560434c11c9e" H 3450 1550 50  0001 L CNN
+	1    3450 1550
+	1    0    0    -1
+$EndComp
+$Comp
+L Transistor_FET:IRF7748L1 Q?
+U 1 1 5AE64A1D
+P 3450 3150
+F 0 "Q?" H 3656 3196 50  0000 L CNN
+F 1 "IRF7748L1" H 3656 3105 50  0000 L CNN
+F 2 "Package_DirectFET:DirectFET_L6" H 3450 3150 50  0001 C CIN
+F 3 "https://www.infineon.com/dgdl/irf7748l1pbf.pdf?fileId=5546d462533600a40153560434c11c9e" H 3450 3150 50  0001 L CNN
+	1    3450 3150
+	1    0    0    -1
+$EndComp
+$Comp
+L Transistor_FET:IRF7748L1 Q?
+U 1 1 5AE64A77
+P 6850 1500
+F 0 "Q?" H 7056 1546 50  0000 L CNN
+F 1 "IRF7748L1" H 7056 1455 50  0000 L CNN
+F 2 "Package_DirectFET:DirectFET_L6" H 6850 1500 50  0001 C CIN
+F 3 "https://www.infineon.com/dgdl/irf7748l1pbf.pdf?fileId=5546d462533600a40153560434c11c9e" H 6850 1500 50  0001 L CNN
+	1    6850 1500
+	1    0    0    -1
+$EndComp
+$Comp
+L Transistor_FET:IRF7748L1 Q?
+U 1 1 5AE64B03
+P 6900 3200
+F 0 "Q?" H 7106 3246 50  0000 L CNN
+F 1 "IRF7748L1" H 7106 3155 50  0000 L CNN
+F 2 "Package_DirectFET:DirectFET_L6" H 6900 3200 50  0001 C CIN
+F 3 "https://www.infineon.com/dgdl/irf7748l1pbf.pdf?fileId=5546d462533600a40153560434c11c9e" H 6900 3200 50  0001 L CNN
+	1    6900 3200
+	1    0    0    -1
+$EndComp
+$Comp
+L Transistor_FET:IRF7748L1 Q?
+U 1 1 5AE64B6D
+P 9750 1500
+F 0 "Q?" H 9956 1546 50  0000 L CNN
+F 1 "IRF7748L1" H 9956 1455 50  0000 L CNN
+F 2 "Package_DirectFET:DirectFET_L6" H 9750 1500 50  0001 C CIN
+F 3 "https://www.infineon.com/dgdl/irf7748l1pbf.pdf?fileId=5546d462533600a40153560434c11c9e" H 9750 1500 50  0001 L CNN
+	1    9750 1500
+	1    0    0    -1
+$EndComp
+$Comp
+L Transistor_FET:IRF7748L1 Q?
+U 1 1 5AE64BD7
+P 9700 3150
+F 0 "Q?" H 9906 3196 50  0000 L CNN
+F 1 "IRF7748L1" H 9906 3105 50  0000 L CNN
+F 2 "Package_DirectFET:DirectFET_L6" H 9700 3150 50  0001 C CIN
+F 3 "https://www.infineon.com/dgdl/irf7748l1pbf.pdf?fileId=5546d462533600a40153560434c11c9e" H 9700 3150 50  0001 L CNN
+	1    9700 3150
+	1    0    0    -1
+$EndComp
 $EndSCHEMATC

Commit message: finish power and can schematic but many components librariy has error
Parts:
- removed Q? (x4): IRF7748L1, Package_DirectFET:DirectFET_L6, symbol Transistor_FET:IRF7748L1
- removed U? (x2): AD8418, symbol Amplifier_Current:AD8418
- added C? (x15): C, symbol Device:C
- added Q? (x4): IRF7748L1, Package_DirectFET:DirectFET_L6, symbol Transistor_FET:IRF7748L1
- added R? (x14): R, symbol Device:R
- added U? (x2): AD8418, symbol Amplifier_Current:AD8418
Connections:
- net labels added: CURR_A, CURR_B, CURR_C, C_A, C_B, C_C, GH_A, GH_B, GH_C, GL_A, GL_B, GL_C, GND, PH_A, PH_B, PH_C, SH_A, SH_B, SH_C, SL_A, SL_B, SL_C, SUPPLY, TEMP, VCC
- wire segments 0 -> 145
Other:
- moved on the sheet: Q?, U?

Commit message: finished schematic and rename LESC to ESCX
Parts:
- added J7: PH_B, symbol Connector_Generic:Conn_01x01
- added J8: PH_A, symbol Connector_Generic:Conn_01x01
- added J9: PH_C, symbol Connector_Generic:Conn_01x01
- gave numbers to parts that had none: 38
Connections:
- net labels removed: PH_A, PH_B, PH_C

Commit message: add value
Parts:
- added J10: GND, symbol Connector_Generic:Conn_01x01
- C29: renamed from C33; value C -> 2.2u
- C30: renamed from C37; value C -> 4.7n
- C31: renamed from C39; value C -> 4.7n
- C32: renamed from C40; value C -> 4.7n
- C33: renamed from C28; value C -> 4.7u_100v
- C34: renamed from C29; value C -> 4.7u_100v
- C35: renamed from C32; value C -> 2.2u
- C36: renamed from C38; value C -> 2.2u
- C37: renamed from C26; value C -> 4.7u_100v
- C38: renamed from C27; value C -> 4.7u_100v
- C39: renamed from C34; value C -> 2.2u
- C40: renamed from C35; value C -> 680u_63v
- C41: renamed from C36; value C -> 680u_63v
- C42: renamed from C30; value C -> 4.7u_100v
- C43: renamed from C31; value C -> 4.7u_100v
- R25: renamed from R29; value R -> 0.0005R
- R26: value R -> 4.7R
- R27: renamed from R32; value R -> 4.7R
- R28: renamed from R34; value R -> 100R
- R29: renamed from R37; value R -> 100R
- R30: renamed from R38; value R -> 100R
- R31: renamed from R28; value R -> 0.005R
- R32: renamed from R35; value R -> NTC 10k
- R33: renamed from R36; value R -> 10k
- R34: renamed from R25; value R -> 4.7R
- R35: renamed from R31; value R -> 4.7R
- R37: renamed from R27; value R -> 4.7R
- R38: renamed from R33; value R -> 4.7R
- renumbered J8 to J7, J7 to J8, Q2 to Q1, Q5 to Q2, Q1 to Q3, Q3 to Q5, R30 to R36, U3 to U5, U5 to U6

Commit message: add bldc lib, link major component to this lib
Parts:
- removed Q1, Q2, Q3, Q4, Q5, Q6: IRF7748L1, Package_DirectFET:DirectFET_L6, symbol Transistor_FET:IRF7748L1
- added J?: SUPPLY, symbol Connector_Generic:Conn_01x01
- added Q? (x6): IRF7749, symbol bldc:IRF7749
Connections:
- wire segments 145 -> 146
Changed lines of the file:
@@
-$EndComp
-$Comp
-L Transistor_FET:IRF7748L1 Q3
-U 1 1 5AE649B5
-P 6600 1600
-F 0 "Q3" H 6806 1646 50  0000 L CNN
-F 1 "IRF7748L1" H 6250 1850 50  0000 L CNN
-F 2 "Package_DirectFET:DirectFET_L6" H 6600 1600 50  0001 C CIN
-F 3 "https://www.infineon.com/dgdl/irf7748l1pbf.pdf?fileId=5546d462533600a40153560434c11c9e" H 6600 1600 50  0001 L CNN
-	1    6600 1600
-	1    0    0    -1
-$EndComp
-$Comp
-L Transistor_FET:IRF7748L1 Q4
-U 1 1 5AE64A1D
-P 6600 3200
-F 0 "Q4" H 6806 3246 50  0000 L CNN
-F 1 "IRF7748L1" H 6300 3400 50  0000 L CNN
-F 2 "Package_DirectFET:DirectFET_L6" H 6600 3200 50  0001 C CIN
-F 3 "https://www.infineon.com/dgdl/irf7748l1pbf.pdf?fileId=5546d462533600a40153560434c11c9e" H 6600 3200 50  0001 L CNN
-	1    6600 3200
-	1    0    0    -1
 $EndComp
 $Comp
@@
 $EndComp
 $Comp
-L Transistor_FET:IRF7748L1 Q1
-U 1 1 5AE2EF36
-P 2900 1650
-F 0 "Q1" H 3106 1696 50  0000 L CNN
-F 1 "IRF7748L1" H 2550 1900 50  0000 L CNN
-F 2 "Package_DirectFET:DirectFET_L6" H 2900 1650 50  0001 C CIN
-F 3 "https://www.infineon.com/dgdl/irf7748l1pbf.pdf?fileId=5546d462533600a40153560434c11c9e" H 2900 1650 50  0001 L CNN
-	1    2900 1650
-	1    0    0    -1
-$EndComp
-$Comp
-L Transistor_FET:IRF7748L1 Q2
-U 1 1 5AE2EF3C
-P 2900 3250
-F 0 "Q2" H 3106 3296 50  0000 L CNN
-F 1 "IRF7748L1" H 2600 3450 50  0000 L CNN
-F 2 "Package_DirectFET:DirectFET_L6" H 2900 3250 50  0001 C CIN
-F 3 "https://www.infineon.com/dgdl/irf7748l1pbf.pdf?fileId=5546d462533600a40153560434c11c9e" H 2900 3250 50  0001 L CNN
-	1    2900 3250
-	1    0    0    -1
-$EndComp
-$Comp
 L Device:R R26
 U 1 1 5AE2EF42
@@
 $EndComp
 $Comp
-L Transistor_FET:IRF7748L1 Q5
-U 1 1 5AE3105F
-P 10050 1650
-F 0 "Q5" H 10256 1696 50  0000 L CNN
-F 1 "IRF7748L1" H 9700 1900 50  0000 L CNN
-F 2 "Package_DirectFET:DirectFET_L6" H 10050 1650 50  0001 C CIN
-F 3 "https://www.infineon.com/dgdl/irf7748l1pbf.pdf?fileId=5546d462533600a40153560434c11c9e" H 10050 1650 50  0001 L CNN
-	1    10050 1650
-	1    0    0    -1
-$EndComp
-$Comp
-L Transistor_FET:IRF7748L1 Q6
-U 1 1 5AE31065
-P 10050 3250
-F 0 "Q6" H 10256 3296 50  0000 L CNN
-F 1 "IRF7748L1" H 9750 3550 50  0000 L CNN
-F 2 "Package_DirectFET:DirectFET_L6" H 10050 3250 50  0001 C CIN
-F 3 "https://www.infineon.com/dgdl/irf7748l1pbf.pdf?fileId=5546d462533600a40153560434c11c9e" H 10050 3250 50  0001 L CNN
-	1    10050 3250
-	1    0    0    -1
-$EndComp
-$Comp
 L Device:R R37
 U 1 1 5AE3106B
@@
 Wire Wire Line
 	10150 1100 10150 1450
-Connection ~ 3000 1450
-Connection ~ 10150 1450
 Wire Wire Line
 	6700 1100 6700 1400
-Connection ~ 6700 1400
 Wire Wire Line
 	3000 4250 6700 4250
@@
 	1    0    0    -1
 $EndComp
+Text HLabel 10150 800  0    50   Input ~ 0
+SUPPLY
+Wire Wire Line
+	10150 800  10150 1100
+Connection ~ 10150 1100
+$Comp
+L Connector_Generic:Conn_01x01 J?
+U 1 1 5B168A48
+P 10350 1100
+F 0 "J?" H 10350 1200 50  0000 C CNN
+F 1 "SUPPLY" H 10350 1000 50  0000 C CNN
+F 2 "" H 10350 1100 50  0001 C CNN
+F 3 "~" H 10350 1100 50  0001 C CNN
+	1    10350 1100
+	1    0    0    -1
+$EndComp
+$Comp
+L bldc:IRF7749 Q?
+U 1 1 5B1C0925
+P 3000 1650
+F 0 "Q?" H 3106 1696 50  0000 L CNN
+F 1 "IRF7749" H 3106 1605 50  0000 L CNN
+F 2 "" H 3000 1650 50  0001 C CNN
+F 3 "" H 3000 1650 50  0001 C CNN
+	1    3000 1650
+	1    0    0    -1
+$EndComp
+Connection ~ 3000 1450
+$Comp
+L bldc:IRF7749 Q?
+U 1 1 5B1C81B4
+P 3000 3250
+F 0 "Q?" H 3106 3296 50  0000 L CNN
+F 1 "IRF7749" H 3106 3205 50  0000 L CNN
+F 2 "" H 3000 3250 50  0001 C CNN
+F 3 "" H 3000 3250 50  0001 C CNN
+	1    3000 3250
+	1    0    0    -1
+$EndComp
+$Comp
+L bldc:IRF7749 Q?
+U 1 1 5B1C8A99
+P 6700 1600
+F 0 "Q?" H 6806 1646 50  0000 L CNN
+F 1 "IRF7749" H 6806 1555 50  0000 L CNN
+F 2 "" H 6700 1600 50  0001 C CNN
+F 3 "" H 6700 1600 50  0001 C CNN
+	1    6700 1600
+	1    0    0    -1
+$EndComp
+Connection ~ 6700 1400
+$Comp
+L bldc:IRF7749 Q?
+U 1 1 5B1C8BE9
+P 6700 3200
+F 0 "Q?" H 6806 3246 50  0000 L CNN
+F 1 "IRF7749" H 6806 3155 50  0000 L CNN
+F 2 "" H 6700 3200 50  0001 C CNN
+F 3 "" H 6700 3200 50  0001 C CNN
+	1    6700 3200
+	1    0    0    -1
+$EndComp
+$Comp
+L bldc:IRF7749 Q?
+U 1 1 5B1C8DFD
+P 10150 3250
+F 0 "Q?" H 10256 3296 50  0000 L CNN
+F 1 "IRF7749" H 10256 3205 50  0000 L CNN
+F 2 "" H 10150 3250 50  0001 C CNN
+F 3 "" H 10150 3250 50  0001 C CNN
+	1    10150 3250
+	1    0    0    -1
+$EndComp
+$Comp
+L bldc:IRF7749 Q?
+U 1 1 5B1C8EF5
+P 10150 1650
+F 0 "Q?" H 10256 1696 50  0000 L CNN
+F 1 "IRF7749" H 10256 1605 50  0000 L CNN
+F 2 "" H 10150 1650 50  0001 C CNN
+F 3 "" H 10150 1650 50  0001 C CNN
+	1    10150 1650
+	1    0    0    -1
+$EndComp
+Connection ~ 10150 1450
 $EndSCHEMATC

Commit message: finish sch
Parts:
- Q1, Q2, Q3, Q4, Q5, Q6: renamed from Q?; footprint (none) -> Package_DirectFET:DirectFET_L8; symbol bldc:IRF7749 -> bldc:IRF7749L1PBF
- R31: value 0.005R -> 0.0005R
- R36: value R -> 0.0005R
- gave numbers to parts that had none: 1
- renumbered C29 to C33, C30 to C34, C31 to C35, C32 to C36, C33 to C37, C34 to C38, C35 to C39, C36 to C40, C37 to C41, C38 to C42, C39 to C43, C40 to C44, C41 to C45, C42 to C46, C43 to C47, J10 to J11
Connections:
- wire segments 146 -> 148
